File: ImogenWren.kicad_pcb (KiCad board)
At the start: 2 copper layers, 85.1 x 53.3 mm, 9 parts

Commit message: n;kln;sfdg
Parts:
- added REF**: PinHeader_1x10_P2.54mm_Vertical, Connector_PinHeader_2.54mm:PinHeader_1x10_P2.54mm_Vertical, F.Cu at (217.2, 71.1)
- added REF**: BUS_PCIexpress_x1, Connector_PCBEdge:BUS_PCIexpress_x1, F.Cu at (143.2, 72.4)
Changed lines of the file:
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@@
       (stroke (width 0) (type solid)) (fill solid) (layer "F.Cu"))
+  )
+  (footprint "Connector_PinHeader_2.54mm:PinHeader_1x10_P2.54mm_Vertical" (layer "F.Cu")
+    (at 217.17 71.12)
+    (descr "Through hole straight pin header, 1x10, 2.54mm pitch, single row")
+    (tags "Through hole pin header THT 1x10 2.54mm single row")
+    (attr through_hole)
+    (fp_text reference "REF**" (at 0 -2.33) (layer "F.SilkS")
+        (effects (font (size 1 1) (thickness 0.15)))
+    )
+    (fp_text value "PinHeader_1x10_P2.54mm_Vertical" (at 0 25.19) (layer "F.Fab")
+        (effects (font (size 1 1) (thickness 0.15)))
+    )
+    (fp_text user "${REFERENCE}" (at 0 11.43 90) (layer "F.Fab")
+        (effects (font (size 1 1) (thickness 0.15)))
+    )
+    (fp_line (start -1.33 -1.33) (end 0 -1.33)
+      (stroke (width 0.12) (type solid)) (layer "F.SilkS"))
+    (fp_line (start -1.33 0) (end -1.33 -1.33)
+      (stroke (width 0.12) (type solid)) (layer "F.SilkS"))
+    (fp_line (start -1.33 1.27) (end -1.33 24.19)
+      (stroke (width 0.12) (type solid)) (layer "F.SilkS"))
+    (fp_line (start -1.33 1.27) (end 1.33 1.27)
+      (stroke (width 0.12) (type solid)) (layer "F.SilkS"))
+    (fp_line (start -1.33 24.19) (end 1.33 24.19)
+      (stroke (width 0.12) (type solid)) (layer "F.SilkS"))
+    (fp_line (start 1.33 1.27) (end 1.33 24.19)
+      (stroke (width 0.12) (type solid)) (layer "F.SilkS"))
+    (fp_line (start -1.8 -1.8) (end -1.8 24.65)
+      (stroke (width 0.05) (type solid)) (layer "F.CrtYd"))
+    (fp_line (start -1.8 24.65) (end 1.8 24.65)
+      (stroke (width 0.05) (type solid)) (layer "F.CrtYd"))
+    (fp_line (start 1.8 -1.8) (end -1.8 -1.8)
+      (stroke (width 0.05) (type solid)) (layer "F.CrtYd"))
+    (fp_line (start 1.8 24.65) (end 1.8 -1.8)
+      (stroke (width 0.05) (type solid)) (layer "F.CrtYd"))
+    (fp_line (start -1.27 -0.635) (end -0.635 -1.27)
+      (stroke (width 0.1) (type solid)) (layer "F.Fab"))
+    (fp_line (start -1.27 24.13) (end -1.27 -0.635)
+      (stroke (width 0.1) (type solid)) (layer "F.Fab"))
+    (fp_line (start -0.635 -1.27) (end 1.27 -1.27)
+      (stroke (width 0.1) (type solid)) (layer "F.Fab"))
+    (fp_line (start 1.27 -1.27) (end 1.27 24.13)
+      (stroke (width 0.1) (type solid)) (layer "F.Fab"))
+    (fp_line (start 1.27 24.13) (end -1.27 24.13)
+      (stroke (width 0.1) (type solid)) (layer "F.Fab"))
+    (pad "1" thru_hole rect (at 0 0) (size 1.7 1.7) (drill 1) (layers "*.Cu" "*.Mask"))
+    (pad "2" thru_hole oval (at 0 2.54) (size 1.7 1.7) (drill 1) (layers "*.Cu" "*.Mask"))
+    (pad "3" thru_hole oval (at 0 5.08) (size 1.7 1.7) (drill 1) (layers "*.Cu" "*.Mask"))
+    (pad "4" thru_hole oval (at 0 7.62) (size 1.7 1.7) (drill 1) (layers "*.Cu" "*.Mask"))
+    (pad "5" thru_hole oval (at 0 10.16) (size 1.7 1.7) (drill 1) (layers "*.Cu" "*.Mask"))
+    (pad "6" thru_hole oval (at 0 12.7) (size 1.7 1.7) (drill 1) (layers "*.Cu" "*.Mask"))
+    (pad "7" thru_hole oval (at 0 15.24) (size 1.7 1.7) (drill 1) (layers "*.Cu" "*.Mask"))
+    (pad "8" thru_hole oval (at 0 17.78) (size 1.7 1.7) (drill 1) (layers "*.Cu" "*.Mask"))
+    (pad "9" thru_hole oval (at 0 20.32) (size 1.7 1.7) (drill 1) (layers "*.Cu" "*.Mask"))
+    (pad "10" thru_hole oval (at 0 22.86) (size 1.7 1.7) (drill 1) (layers "*.Cu" "*.Mask"))
+    (model "${KICAD6_3DMODEL_DIR}/Connector_PinHeader_2.54mm.3dshapes/PinHeader_1x10_P2.54mm_Vertical.wrl"
+      (offset (xyz 0 0 0))
+      (scale (xyz 1 1 1))
+      (rotate (xyz 0 0 0))
+    )
   )
   (footprint "000_Graphics_Immo:cu_heart" (layer "F.Cu")
@@
     (pad "" np_thru_hole circle (at 0 0) (size 3.2 3.2) (drill 3.2) (layers "*.Cu" "*.Mask"))
   )
+  (footprint "Connector_PCBEdge:BUS_PCIexpress_x1" (layer "F.Cu")
+    (at 143.24 72.39 180)
+    (descr "PCIexpress Bus Edge Connector x1 http://www.ritrontek.com/uploadfile/2016/1026/20161026105231124.pdf#page=70")
+    (tags "PCIe")
+    (attr exclude_from_pos_files exclude_from_bom)
+    (fp_text reference "REF**" (at 5 -3.5) (layer "F.SilkS")
+        (effects (font (size 1 1) (thickness 0.15)))
+    )
+    (fp_text value "BUS_PCIexpress_x1" (at 10.33 -8.01) (layer "F.Fab")
+        (effects (font (size 1 1) (thickness 0.15)))
+    )
+    (fp_text user "PCB Thickness 1.57 mm" (at 5 2.8) (layer "Cmts.User")
+        (effects (font (size 0.5 0.5) (thickness 0.1)))
+    )
+    (fp_text user "${REFERENCE}" (at 16 -3.5) (layer "F.Fab")
+        (effects (font (size 1 1) (thickness 0.15)))
+    )
+    (fp_line (start -0.65 -4.95) (end -0.65 2.95)
+      (stroke (width 0.1) (type solid)) (layer "Edge.Cuts"))
+    (fp_line (start -0.65 2.95) (end -0.15 3.45)
+      (stroke (width 0.1) (type solid)) (layer "Edge.Cuts"))
+    (fp_line (start -0.15 3.45) (end 10.05 3.45)
+      (stroke (width 0.1) (type solid)) (layer "Edge.Cuts"))
+    (fp_line (start 10.55 -4) (end 10.55 2.95)
+      (stroke (width 0.1) (type solid)) (layer "Edge.Cuts"))
+    (fp_line (start 10.55 2.95) (end 10.05 3.45)
+      (stroke (width 0.1) (type solid)) (layer "Edge.Cuts"))
+    (fp_line (start 12.45 -4) (end 12.45 2.95)
+      (stroke (width 0.1) (type solid)) (layer "Edge.Cuts"))
+    (fp_line (start 12.45 2.95) (end 12.95 3.45)
+      (stroke (width 0.1) (type solid)) (layer "Edge.Cuts"))
+    (fp_line (start 12.95 3.45) (end 19.15 3.45)
+      (stroke (width 0.1) (type solid)) (layer "Edge.Cuts"))
+    (fp_line (start 19.65 -4.95) (end 19.65 2.95)
+      (stroke (width 0.1) (type solid)) (layer "Edge.Cuts"))
+    (fp_line (start 19.65 2.95) (end 19.15 3.45)
+      (stroke (width 0.1) (type solid)) (layer "Edge.Cuts"))
+    (fp_arc (start 10.55 -4) (mid 11.5 -4.95) (end 12.45 -4)
+      (stroke (width 0.1) (type solid)) (layer "Edge.Cuts"))
+    (fp_line (start -1.15 -5.45) (end -1.15 3.95)
+      (stroke (width 0.05) (type solid)) (layer "F.CrtYd"))
+    (fp_line (start -1.15 -5.45) (end 20.15 -5.45)
+      (stroke (width 0.05) (type solid)) (layer "F.CrtYd"))
+    (fp_line (start 20.15 3.95) (end -1.15 3.95)
+      (stroke (width 0.05) (type solid)) (layer "F.CrtYd"))
+    (fp_line (start 20.15 3.95) (end 20.15 -5.45)
+      (stroke (width 0.05) (type solid)) (layer "F.CrtYd"))
+    (pad "A1" connect rect (at 0 -0.55 180) (size 0.7 3.2) (layers "B.Cu" "B.Mask"))
+    (pad "A2" connect rect (at 1 0 180) (size 0.7 4.3) (layers "B.Cu" "B.Mask"))
+    (pad "A3" connect rect (at 2 0 180) (size 0.7 4.3) (layers "B.Cu" "B.Mask"))
+    (pad "A4" connect rect (at 3 0 180) (size 0.7 4.3) (layers "B.Cu" "B.Mask"))
+    (pad "A5" connect rect (at 4 0 180) (size 0.7 4.3) (layers "B.Cu" "B.Mask"))
+    (pad "A6" connect rect (at 5 0 180) (size 0.7 4.3) (layers "B.Cu" "B.Mask"))
+    (pad "A7" connect rect (at 6 0 180) (size 0.7 4.3) (layers "B.Cu" "B.Mask"))
+    (pad "A8" connect rect (at 7 0 180) (size 0.7 4.3) (layers "B.Cu" "B.Mask"))
+    (pad "A9" connect rect (at 8 0 180) (size 0.7 4.3) (layers "B.Cu" "B.Mask"))
+    (pad "A10" connect rect (at 9 0 180) (size 0.7 4.3) (layers "B.Cu" "B.Mask"))
+    (pad "A11" connect rect (at 10 0 180) (size 0.7 4.3) (layers "B.Cu" "B.Mask"))
+    (pad "A12" connect rect (at 13 0 180) (size 0.7 4.3) (layers "B.Cu" "B.Mask"))
+    (pad "A13" connect rect (at 14 0 180) (size 0.7 4.3) (layers "B.Cu" "B.Mask"))
+    (pad "A14" connect rect (at 15 0 180) (size 0.7 4.3) (layers "B.Cu" "B.Mask"))
+    (pad "A15" connect rect (at 16 0 180) (size 0.7 4.3) (layers "B.Cu" "B.Mask"))
+    (pad "A16" connect rect (at 17 0 180) (size 0.7 4.3) (layers "B.Cu" "B.Mask"))
+    (pad "A17" connect rect (at 18 0 180) (size 0.7 4.3) (layers "B.Cu" "B.Mask"))
+    (pad "A18" connect rect (at 19 0 180) (size 0.7 4.3) (layers "B.Cu" "B.Mask"))
+    (pad "B1" connect rect (at 0 0 180) (size 0.7 4.3) (layers "F.Cu" "F.Mask"))
+    (pad "B2" connect rect (at 1 0 180) (size 0.7 4.3) (layers "F.Cu" "F.Mask"))
+    (pad "B3" connect rect (at 2 0 180) (size 0.7 4.3) (layers "F.Cu" "F.Mask"))
+    (pad "B4" connect rect (at 3 0 180) (size 0.7 4.3) (layers "F.Cu" "F.Mask"))
+    (pad "B5" connect rect (at 4 0 180) (size 0.7 4.3) (layers "F.Cu" "F.Mask"))
+    (pad "B6" connect rect (at 5 0 180) (size 0.7 4.3) (layers "F.Cu" "F.Mask"))
+    (pad "B7" connect rect (at 6 0 180) (size 0.7 4.3) (layers "F.Cu" "F.Mask"))
+    (pad "B8" connect rect (at 7 0 180) (size 0.7 4.3) (layers "F.Cu" "F.Mask"))
+    (pad "B9" connect rect (at 8 0 180) (size 0.7 4.3) (layers "F.Cu" "F.Mask"))
+    (pad "B10" connect rect (at 9 0 180) (size 0.7 4.3) (layers "F.Cu" "F.Mask"))
+    (pad "B11" connect rect (at 10 0 180) (size 0.7 4.3) (layers "F.Cu" "F.Mask"))
+    (pad "B12" connect rect (at 13 0 180) (size 0.7 4.3) (layers "F.Cu" "F.Mask"))
+    (pad "B13" connect rect (at 14 0 180) (size 0.7 4.3) (layers "F.Cu" "F.Mask"))
+    (pad "B14" connect rect (at 15 0 180) (size 0.7 4.3) (layers "F.Cu" "F.Mask"))
+    (pad "B15" connect rect (at 16 0 180) (size 0.7 4.3) (layers "F.Cu" "F.Mask"))
+    (pad "B16" connect rect (at 17 0 180) (size 0.7 4.3) (layers "F.Cu" "F.Mask"))
+    (pad "B17" connect rect (at 18 -0.55 180) (size 0.7 3.2) (layers "F.Cu" "F.Mask"))
+    (pad "B18" connect rect (at 19 0 180) (size 0.7 4.3) (layers "F.Cu" "F.Mask"))
+  )
   (footprint "000_Graphics_Immo:ImogenWren70_Cu" (layer "F.Cu")

Commit message: kjsaofklihsdof
Parts:
- removed the REF** at (217.2, 71.1)
- added BT1: Battery_Cell, Battery:BatteryHolder_Keystone_1060_1x2032, B.Cu at (104.1, 22.6)
- added C1: 100n, Capacitor_SMD:C_0805_2012Metric_Pad1.18x1.45mm_HandSolder, B.Cu at (40.0, 138.8)
- added C10: 100n, Capacitor_SMD:C_0805_2012Metric_Pad1.18x1.45mm_HandSolder, B.Cu at (-3.85, 63.8)
- added C11: 47p, Capacitor_SMD:C_0805_2012Metric_Pad1.18x1.45mm_HandSolder, B.Cu at (-3.85, 66.8)
- added C12: 4n7, Capacitor_SMD:C_0805_2012Metric_Pad1.18x1.45mm_HandSolder, B.Cu at (-3.85, 69.8)
- added C13: 100n, Capacitor_SMD:C_0805_2012Metric_Pad1.18x1.45mm_HandSolder, B.Cu at (164.4, 150.1)
- added C14: 100n, Capacitor_SMD:C_0805_2012Metric_Pad1.18x1.45mm_HandSolder, B.Cu at (28.8, 124.3)
- added C15: 100n, Capacitor_SMD:C_0805_2012Metric_Pad1.18x1.45mm_HandSolder, B.Cu at (28.8, 127.3)
- added C16: 100n, Capacitor_SMD:C_0805_2012Metric_Pad1.18x1.45mm_HandSolder, B.Cu at (28.8, 130.3)
- added C17: 100n, Capacitor_SMD:C_0805_2012Metric_Pad1.18x1.45mm_HandSolder, B.Cu at (159.6, 150.1)
- added C18: 100n, Capacitor_SMD:C_0805_2012Metric_Pad1.18x1.45mm_HandSolder, B.Cu at (24.0, 124.3)
- added C19: 100n, Capacitor_SMD:C_0805_2012Metric_Pad1.18x1.45mm_HandSolder, B.Cu at (24.0, 127.3)
- added C2: 100n, Capacitor_SMD:C_0805_2012Metric_Pad1.18x1.45mm_HandSolder, B.Cu at (159.0, 38.0)
- added C20: 100n, Capacitor_SMD:C_0805_2012Metric_Pad1.18x1.45mm_HandSolder, B.Cu at (24.0, 130.3)
- added C21: 100n, Capacitor_SMD:C_0805_2012Metric_Pad1.18x1.45mm_HandSolder, B.Cu at (154.7, 150.1)
- added C22: 100n, Capacitor_SMD:C_0805_2012Metric_Pad1.18x1.45mm_HandSolder, B.Cu at (19.2, 124.3)
- added C23: 100n, Capacitor_SMD:C_0805_2012Metric_Pad1.18x1.45mm_HandSolder, B.Cu at (19.2, 127.3)
- added C24: 100n, Capacitor_SMD:C_0805_2012Metric_Pad1.18x1.45mm_HandSolder, B.Cu at (19.2, 130.3)
- added C3: 100n, Capacitor_SMD:C_0805_2012Metric_Pad1.18x1.45mm_HandSolder, B.Cu at (159.0, 41.0)
- added C4: 100n, Capacitor_SMD:C_0805_2012Metric_Pad1.18x1.45mm_HandSolder, B.Cu at (159.0, 44.0)
- added C5: 100n, Capacitor_SMD:C_0805_2012Metric_Pad1.18x1.45mm_HandSolder, B.Cu at (159.0, 47.0)
- added C6: 100n, Capacitor_SMD:C_0805_2012Metric_Pad1.18x1.45mm_HandSolder, B.Cu at (144.0, 52.3)
- added C7: 100n, Capacitor_SMD:C_0805_2012Metric_Pad1.18x1.45mm_HandSolder, B.Cu at (144.0, 55.3)
- added C8: 10n, Capacitor_SMD:C_0805_2012Metric_Pad1.18x1.45mm_HandSolder, B.Cu at (-3.85, 57.7)
- added C9: 47p, Capacitor_SMD:C_0805_2012Metric_Pad1.18x1.45mm_HandSolder, B.Cu at (-3.85, 60.8)
- added D1: Blue, LED_SMD:LED_0805_2012Metric_Pad1.15x1.40mm_HandSolder, B.Cu at (149.4, 46.3)
- added EC1: 1000u, Capacitor_SMD:CP_Elec_10x10, B.Cu at (64.6, 128.3)
- added FB1: FerriteBead, Inductor_SMD:L_0805_2012Metric_Pad1.05x1.20mm_HandSolder, B.Cu at (-8.70, 68.1)
- added J1: WS2821_LED_OUT, Connector_PCBEdge:BUS_PCIexpress_x1, B.Cu at (138.5, 117.6)
- added J2: SDI/SDO, Connector_PCBEdge:BUS_PCIexpress_x1, B.Cu at (119.4, 71.8)
- added J3: ESP_GPIO_B, Connector_PCBEdge:BUS_PCIexpress_x1, B.Cu at (207.2, 154.6)
- added J4: ESPpin4-7, Connector_PCBEdge:BUS_PCIexpress_x1, B.Cu at (223.6, 136.6)
- added J5: 1-pin-edge-touch-XL, Connector_PCBEdge:BUS_PCIexpress_x1, B.Cu at (185.5, 107.3)
- added J6: Touch Pins, 000-edge-connectors-immo:8-pin-edge-touch, B.Cu at (178.2, 117.9)
- added J7: i2c Header, Connector_PCBEdge:BUS_PCIexpress_x1, B.Cu at (168.9, 71.9)
- added J8: USB_C_Receptacle, Connector_USB:USB_C_Receptacle_Molex_105450-0101, B.Cu at (116.0, 94.6)
- added JP1: I Prog, Jumper:SolderJumper-3_P1.3mm_Open_RoundedPad1.0x1.5mm_NumberLabels, B.Cu at (64.8, 136.0)
- added JP2: Power Routing, Jumper:SolderJumper-3_P1.3mm_Bridged12_RoundedPad1.0x1.5mm, B.Cu at (55.0, 134.6)
- added JP3: LED_DATA_SOURCE, Jumper:SolderJumper-3_P1.3mm_Bridged12_RoundedPad1.0x1.5mm, B.Cu at (55.0, 138.4)
- added JPw1: Disable Onboard LEDs, Jumper:SolderJumper-2_P1.3mm_Bridged_RoundedPad1.0x1.5mm, B.Cu at (69.8, 136.0)
- added Q1: BC817, Package_TO_SOT_SMD:SOT-23, B.Cu at (135.5, 51.7)
- added Q2: BC817, Package_TO_SOT_SMD:SOT-23, B.Cu at (135.5, 56.1)
- added R1: 10k, Resistor_SMD:R_0805_2012Metric_Pad1.20x1.40mm_HandSolder, B.Cu at (35.6, 101.4)
- added R10: 10k, Resistor_SMD:R_0805_2012Metric_Pad1.20x1.40mm_HandSolder, B.Cu at (130.7, 50.9)
- added R11: 10k, Resistor_SMD:R_0805_2012Metric_Pad1.20x1.40mm_HandSolder, B.Cu at (130.7, 53.9)
- added R12: 5k2, Resistor_SMD:R_0805_2012Metric_Pad1.20x1.40mm_HandSolder, B.Cu at (-13.5, 68.2)
- added R2: 10k, Resistor_SMD:R_0805_2012Metric_Pad1.20x1.40mm_HandSolder, B.Cu at (35.6, 104.4)
- added R3: 4k7, Resistor_SMD:R_0805_2012Metric_Pad1.20x1.40mm_HandSolder, B.Cu at (35.6, 107.3)
- added R4: 27r, Resistor_SMD:R_0805_2012Metric_Pad1.20x1.40mm_HandSolder, B.Cu at (35.6, 110.3)
- added R5: 27r, Resistor_SMD:R_0805_2012Metric_Pad1.20x1.40mm_HandSolder, B.Cu at (35.6, 113.2)
- added R6: 470r, Resistor_SMD:R_0805_2012Metric_Pad1.20x1.40mm_HandSolder, B.Cu at (35.6, 116.2)
- added R7: 330r, Resistor_SMD:R_0805_2012Metric_Pad1.20x1.40mm_HandSolder, B.Cu at (154.2, 46.2)
- added R8: 10k, Resistor_SMD:R_0805_2012Metric_Pad1.20x1.40mm_HandSolder, B.Cu at (154.2, 49.2)
- added R9: 10k, Resistor_SMD:R_0805_2012Metric_Pad1.20x1.40mm_HandSolder, B.Cu at (154.2, 52.1)
- added SW1: Power, Button_Switch_SMD:SW_SPDT_PCM12, B.Cu at (166.5, 19.4)
- added SW2: BOOT, Button_Switch_SMD:SW_SPST_EVQPE1, B.Cu at (133.5, 41.9)
- added SW3: EN, Button_Switch_SMD:SW_SPST_EVQPE1, B.Cu at (133.5, 46.9)
- added U1: MCP73831-2-OT, Package_TO_SOT_SMD:SOT-23-5, B.Cu at (39.8, 135.1)
- added U2: AMS1117-3.3, Package_TO_SOT_SMD:SOT-223-3_TabPin2, B.Cu at (151.7, 40.6)
- added U3: ESP32-WROOM-32, RF_Module:ESP32-WROOM-32, B.Cu at (181.0, 95.1)
- added U4: CH340C, Package_SO:SOIC-16_3.9x9.9mm_P1.27mm, B.Cu at (142.2, 45.1)
- added WLED1: WS2812B, LED_SMD:LED_WS2812B_PLCC4_5.0x5.0mm_P3.2mm, B.Cu at (161.3, 94.6)
- added WLED10: WS2812B, LED_SMD:LED_WS2812B_PLCC4_5.0x5.0mm_P3.2mm, B.Cu at (144.8, 111.1)
- added WLED11: WS2812B, LED_SMD:LED_WS2812B_PLCC4_5.0x5.0mm_P3.2mm, B.Cu at (153.0, 108.9)
- added WLED12: WS2812B, LED_SMD:LED_WS2812B_PLCC4_5.0x5.0mm_P3.2mm, B.Cu at (159.1, 102.8)
- added WLED2: WS2812B, LED_SMD:LED_WS2812B_PLCC4_5.0x5.0mm_P3.2mm, B.Cu at (159.1, 86.4)
- added WLED3: WS2812B, LED_SMD:LED_WS2812B_PLCC4_5.0x5.0mm_P3.2mm, B.Cu at (153.0, 80.3)
- added WLED4: WS2812B, LED_SMD:LED_WS2812B_PLCC4_5.0x5.0mm_P3.2mm, B.Cu at (144.8, 78.1)
- added WLED5: WS2812B, LED_SMD:LED_WS2812B_PLCC4_5.0x5.0mm_P3.2mm, B.Cu at (136.5, 80.3)
- added WLED6: WS2812B, LED_SMD:LED_WS2812B_PLCC4_5.0x5.0mm_P3.2mm, B.Cu at (130.5, 86.4)
- added WLED7: WS2812B, LED_SMD:LED_WS2812B_PLCC4_5.0x5.0mm_P3.2mm, B.Cu at (128.3, 94.6)
- added WLED8: WS2812B, LED_SMD:LED_WS2812B_PLCC4_5.0x5.0mm_P3.2mm, B.Cu at (130.5, 102.9)
- added WLED9: WS2812B, LED_SMD:LED_WS2812B_PLCC4_5.0x5.0mm_P3.2mm, B.Cu at (136.6, 108.9)
- moved REF** 103.9 mm to (243.7, 99.1)
- moved REF** 0.10 mm to (115.5, 71.8)

Commit message: ;j;lkjh;k
Parts:
- J5: footprint Connector_PCBEdge:BUS_PCIexpress_x1 -> 000-edge-connectors-immo:1-pin-edge-touch-xl
- moved C24 135.4 mm to (151.3, 100.5)
- moved C23 130.3 mm to (147.6, 104.8)
- moved C14 127.2 mm to (151.3, 89.6), turned to 90 degrees
- moved C15 124.7 mm to (146.1, 84.7)
- moved C22 123.1 mm to (141.1, 107.2)
- moved C16 122.1 mm to (141.0, 82.0)
- moved C18 112.6 mm to (131.0, 89.0)
- moved C20 110.8 mm to (130.8, 100.8)
- moved C19 109.5 mm to (128.5, 94.5), turned to -90 degrees
- moved SW1 101.0 mm to (145.0, 118.0), turned to 180 degrees
- moved JPw1 89.6 mm to (149.4, 94.7), turned to 0 degrees
- moved EC1 83.4 mm to (141.0, 94.9)
- moved SW3 74.6 mm to (156.5, 117.9)
- moved R11 74.3 mm to (169.2, 117.5)
- moved U2 70.6 mm to (165.0, 110.0)
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
Commit message: xcfgdfgd
Parts:
- removed BT1: Battery_Cell, Battery:BatteryHolder_Keystone_1060_1x2032
- removed J7: i2c Header, Connector_PCBEdge:BUS_PCIexpress_x1
- removed the REF** at (243.7, 99.1)
- added J10: ESPpin1-4, 000-edge-connectors-immo:4-pin-edge, B.Cu at (188.0, 118.1)
- added J9: i2c-header, 000-edge-connectors-immo:5-pin-edge-touch, B.Cu at (178.2, 71.3)
- J1: value WS2821_LED_OUT -> Battery Cell 4.2v; footprint Connector_PCBEdge:BUS_PCIexpress_x1 -> 000-edge-connectors-immo:2-pin-edge
- J2: footprint Connector_PCBEdge:BUS_PCIexpress_x1 -> 000-edge-connectors-immo:6-pin-edge-touch
- J3: value ESP_GPIO_B -> WS2821b-LED-Out; footprint Connector_PCBEdge:BUS_PCIexpress_x1 -> 000-edge-connectors-immo:3-pin-edge
- J4: value ESPpin4-7 -> ESP-gpio-B; footprint Connector_PCBEdge:BUS_PCIexpress_x1 -> 000-edge-connectors-immo:5-pin-edge-touch
- SW1: value Power -> SW_SPDT_small; footprint Button_Switch_SMD:SW_SPDT_PCM12 -> 000_Switches_Immo:SW_SPDT_PCM12
- moved U1 86.5 mm to (122.7, 110.2)
- moved JP3 73.8 mm to (121.9, 105.7), turned to -90 degrees
- moved J4 71.5 mm to (184.6, 71.3), turned to 0 degrees
- moved J3 60.3 mm to (115.1, 107.3), turned to 90 degrees
- moved J1 36.2 mm to (115.1, 110.4), turned to 90 degrees
- moved J2 33.0 mm to (152.4, 71.8)
- moved R9 31.8 mm to (180.6, 78.1)
- moved SW1 21.1 mm to (123.9, 118.1)
- moved U4 15.9 mm to (129.5, 72.3), turned to -90 degrees
- moved R8 11.9 mm to (176.8, 78.1), turned to 0 degrees
- moved Q2 11.3 mm to (171.1, 108.9)
- moved R11 10.2 mm to (174.6, 108.9), turned to -90 degrees
- moved C3 9.59 mm to (165.5, 100.3), turned to 0 degrees
- moved C7 9.48 mm to (120.0, 70.1), turned to -90 degrees
- moved J5 8.76 mm to (178.4, 118.1)
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Connections:
- D1 pad 2: Net-(D1-A) -> 23
- J1 pad A1: (no net) -> GNDPWR
- J1 pad A2: (no net) -> Net-(SW1-B)
- J3 pad A1: (no net) -> Net-(JP3-C)
- J3 pad A2: (no net) -> /BATTERY_POWER_BUS
- J3 pad A3: (no net) -> GND
- J4 pad A1: (no net) -> GND
- J4 pad A2: (no net) -> /ESP32/3V3_BUS
- J4 pad A3: (no net) -> 18
- J4 pad A4: (no net) -> 19
- J4 pad A5: (no net) -> 23
- JP3 pad 2: Net-(J1-Pin_3) -> Net-(JP3-C)
- SW1 pad 2: Net-(BT1-+) -> Net-(SW1-B)
- SW1 pad 3: (no net) -> unconnected-(SW1-C-Pad3)
- U3 pad 30: unconnected-(U3-GPIO18-Pad30) -> 18
- U3 pad 37: Net-(D1-A) -> 23
