File: ImogenWren.kicad_pcb (KiCad board)
At the start: 2 copper layers, 85.1 x 53.3 mm, 82 parts, among them J1 Battery Cell 4.2v, J10 ESPpin1-4, J2 SDI/SDO, J3 WS2821b-LED-Out, J4 ESP-gpio-B, J5 1-pin-edge-touch-XL, J6 Touch Pins, J8 USB_C_Receptacle, J9 i2c-header, Q1 BC817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

Commit message: desgfdfg
Parts:
- moved C10 136.2 mm to (122.8, 113.9), turned to 0 degrees
- moved R12 133.1 mm to (118.6, 83.7), turned to 0 degrees
- moved R6 129.9 mm to (163.3, 92.3), turned to 0 degrees
- moved FB1 127.3 mm to (114.0, 101.9)
- moved C11 124.0 mm to (118.5, 87.0)
- moved C1 121.9 mm to (158.0, 108.2)
- moved C8 121.2 mm to (113.8, 87.0)
- moved C9 120.0 mm to (113.9, 84.1)
- moved C12 118.3 mm to (113.9, 80.8)
- moved R4 105.3 mm to (131.2, 66.0)
- moved R5 103.1 mm to (127.3, 66.0)
- moved R2 100.5 mm to (135.4, 116.3), turned to -90 degrees
- moved R1 98.4 mm to (132.8, 116.3), turned to -90 degrees
- moved R3 95.0 mm to (130.2, 116.3), turned to -90 degrees
- moved JP1 70.2 mm to (133.0, 119.7)
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
Commit message: dfhdyhdre
Parts:
- D1: footprint LED_SMD:LED_0805_2012Metric_Pad1.15x1.40mm_HandSolder -> 000_Diodes_Immo:LED_0805_2012_Kawaii
- EC1: footprint Capacitor_SMD:CP_Elec_10x10 -> 000_Capacitors_Immo:CP_Elec_10x10_kawaii
- J1: value Battery Cell 4.2v -> Battery Cell 4V2
- J3: value WS2821b-LED-Out -> WS2821b
- JP2: value Power Routing -> Batt/USB
- JP3: value LED_DATA_SOURCE -> Pre/Post
- JPw1: value Disable Onboard LEDs -> WL-power
- REF**: footprint 000 Modules Immo:CreditCard -> 000_Modules_Immo:CreditCard
- U1: value MCP73831-2-OT -> MCP73831
- WLED1, WLED10, WLED11, WLED12, WLED2, WLED3, WLED4, WLED5, WLED6, WLED7, WLED8, WLED9: footprint LED_SMD:LED_WS2812B_PLCC4_5.0x5.0mm_P3.2mm -> 000_Modules_Immo:LED_WS2812B_PLCC4_5.0x5.0mm_P3.2mm
- moved R11 28.0 mm to (171.3, 81.0)
- moved C12 21.8 mm to (117.7, 102.2), turned to 90 degrees
- moved C2 20.1 mm to (148.1, 118.3), turned to -90 degrees
- moved J2 18.0 mm to (170.4, 70.6)
- moved C1 16.7 mm to (144.7, 118.3), turned to -90 degrees
- moved U2 16.0 mm to (155.5, 117.3), turned to 0 degrees
- moved C3 13.9 mm to (162.8, 117.2), turned to 90 degrees
- moved SW1 13.2 mm to (137.1, 118.0)
- moved R6 11.5 mm to (165.8, 81.2)
- moved R4 10.5 mm to (121.7, 70.5)
- moved Q1 9.96 mm to (167.3, 86.0), turned to 0 degrees
- moved C11 9.94 mm to (116.7, 77.2)
- moved R5 9.57 mm to (121.7, 73.8)
- moved SW3 9.42 mm to (164.1, 111.1)
- moved JP1 7.74 mm to (129.4, 112.8)
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Other:
- outline, holes or cut-outs redrawn
