File: ImogenWren.kicad_pcb (KiCad board)
At the start: 2 copper layers, 85.1 x 53.3 mm, 82 parts, among them J1 Battery Cell 4V2, J10 ESPpin1-4, J2 SDI/SDO, J3 WS2821b, J4 ESP-gpio-B, J5 1-pin-edge-touch-XL, J6 Touch Pins, J8 USB_C_Receptacle, J9 i2c-header, Q1 BC817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

Commit message: DSGFDSF
Parts:
- added REF**: MountingHole_3.2mm_M3, MountingHole:MountingHole_3.2mm_M3, F.Cu at (142.7, 60.2)
- added REF**: MountingHole_2.2mm_M2, MountingHole:MountingHole_2.2mm_M2, F.Cu at (151.9, 101.4)
- added REF**: MountingHole_2.2mm_M2, MountingHole:MountingHole_2.2mm_M2, F.Cu at (151.9, 88.6)
- added REF**: MountingHole_2.2mm_M2, MountingHole:MountingHole_2.2mm_M2, F.Cu at (139.1, 88.6)
- added REF**: MountingHole_2.2mm_M2, MountingHole:MountingHole_2.2mm_M2, F.Cu at (139.1, 101.4)
- moved Q2 26.6 mm to (176.2, 80.8), turned to 0 degrees
- moved R6 8.65 mm to (167.4, 89.7)
- moved Q1 5.77 mm to (164.8, 80.9)
- moved R10 3.81 mm to (171.6, 80.8), turned to -90 degrees
- moved R11 3.06 mm to (168.3, 80.8)
- moved J10 2.54 mm to (185.6, 117.9)
- moved C3 1.96 mm to (163.8, 115.6)
- moved SW3 1.31 mm to (162.8, 111.0)
- moved J6 0.53 mm to (176.7, 118.6)
- moved R8 0.51 mm to (180.0, 80.9)
- moved SW2 0.40 mm to (162.8, 75.8)
- moved R9 0.39 mm to (183.3, 80.8)
- moved J5 0.33 mm to (181.2, 118.6)
- moved U2 0.15 mm to (155.6, 117.5)

Commit message: cgfhfhfg
Parts:
- removed the REF** at (142.7, 60.2)
- added REF**: MountingHole_2.2mm_M2, MountingHole:MountingHole_2.2mm_M2, F.Cu at (167.1, 94.7)
- added REF**: MountingHole_2.2mm_M2, MountingHole:MountingHole_2.2mm_M2, F.Cu at (144.3, 117.5)
- added REF**: MountingHole_2.2mm_M2, MountingHole:MountingHole_2.2mm_M2, F.Cu at (121.5, 94.7)
- added REF**: MountingHole_2.2mm_M2, MountingHole:MountingHole_2.2mm_M2, F.Cu at (144.3, 71.9)
- C1, C10, C11, C12, C13, C14, C15, C16, C17, C18, C19, C2, C20, C21, C22, C23, C24, C3, C4, C5, C6, C7, C8, C9: footprint Capacitor_SMD:C_0805_2012Metric_Pad1.18x1.45mm_HandSolder -> 000_Capacitors_Immo:C_0805_2012_HandSolder_kawaii
- U3: value ESP32-WROOM-32 -> ESP32-WROOM-32_KAWAII; footprint RF_Module:ESP32-WROOM-32 -> 000_Modules_Immo:ESP32-WROOM-32_KAWAII
- moved C6 19.5 mm to (138.8, 71.5), turned to -90 degrees
- moved R6 15.3 mm to (153.0, 94.8), turned to 90 degrees
- moved J8 11.4 mm to (116.3, 83.4)
- moved R4 10.8 mm to (129.4, 78.1), turned to -90 degrees
- moved C12 10.7 mm to (116.4, 91.6)
- moved FB1 10.6 mm to (113.3, 91.7)
- moved C11 10.1 mm to (126.7, 78.1), turned to 90 degrees
- moved C9 9.42 mm to (122.0, 73.1), turned to 0 degrees
- moved C8 8.20 mm to (118.8, 76.3), turned to 0 degrees
- moved SW2 8.01 mm to (167.1, 82.6), turned to 90 degrees
- moved C1 7.15 mm to (151.8, 117.9)
- moved C2 6.43 mm to (154.5, 117.9)
- moved C3 6.04 mm to (163.6, 109.5)
- moved SW3 5.70 mm to (167.2, 107.4), turned to 90 degrees
- moved U2 5.53 mm to (160.9, 116.3)
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
Commit message: 34terg
Parts:
- added D2: BZV55B3V3, 000_Diodes_Immo:D_MiniMELF_kawaii, B.Cu at (156.8, 69.8)
- added D3: BZV55B3V3, 000_Diodes_Immo:D_MiniMELF_kawaii, B.Cu at (156.8, 73.2)
- added J7: DAC/ADC, 000-edge-connectors-immo:4-pin-edge, B.Cu at (164.2, 71.4)
- added R13: 220r, Resistor_SMD:R_0805_2012Metric_Pad1.20x1.40mm_HandSolder, B.Cu at (159.3, 77.3)
- added R14: 220r, Resistor_SMD:R_0805_2012Metric_Pad1.20x1.40mm_HandSolder, B.Cu at (162.4, 80.2)
- added R15: 100r, Resistor_SMD:R_0805_2012Metric_Pad1.20x1.40mm_HandSolder, B.Cu at (151.1, 73.2)
- added R16: 100r, Resistor_SMD:R_0805_2012Metric_Pad1.20x1.40mm_HandSolder, B.Cu at (151.0, 70.0)
- added REF**: MountingHole_2.1mm_1, 000_mechanical_immo:MountingHole_2.1mm_1, F.Cu at (113.0, 98.8)
- added REF**: MountingHole_2.1mm_1, 000_mechanical_immo:MountingHole_2.1mm_1, F.Cu at (113.0, 108.4)
- added REF**: MountingHole_2.1mm_1, 000_mechanical_immo:MountingHole_2.1mm_1, F.Cu at (166.2, 120.2)
- added REF**: MountingHole_2.1mm_1, 000_mechanical_immo:MountingHole_2.1mm_1, F.Cu at (183.9, 120.2)
- added REF**: MountingHole_2.1mm_1, 000_mechanical_immo:MountingHole_2.1mm_1, F.Cu at (181.1, 120.2)
- added REF**: MountingHole_2.1mm_1, 000_mechanical_immo:MountingHole_2.1mm_1, F.Cu at (176.7, 120.2)
- added REF**: MountingHole_2.1mm_1, 000_mechanical_immo:MountingHole_2.1mm_1, F.Cu at (113.0, 103.2)
- added REF**: MountingHole_2.1mm_1, 000_mechanical_immo:MountingHole_2.1mm_1, F.Cu at (189.6, 120.2)
- added REF**: MountingHole_2.1mm_1, 000_mechanical_immo:MountingHole_2.1mm_1, F.Cu at (113.0, 112.9)
- J1: value Battery Cell 4V2 -> Battery Cell
- J4: value ESP-gpio-B -> gpio-B
- J5: value 1-pin-edge-touch-XL -> Touch0
- JP2: value Batt/USB -> usb/batt
- JP3: value Pre/Post -> led-data
- JPw1: value WL-power -> led-pwr
- U1: value MCP73831 -> MCP73831-2-OT
- U3: value ESP32-WROOM-32_KAWAII -> ESP32-WROOM-32
- moved JP3 21.7 mm to (144.4, 103.0), turned to 0 degrees
- moved C7 14.9 mm to (137.4, 73.3), turned to 0 degrees
- moved Q1 13.5 mm to (167.6, 89.2)
- moved C10 8.05 mm to (122.6, 119.8), turned to 0 degrees
- moved C12 7.13 mm to (122.3, 87.6)
- moved J3 3.99 mm to (118.4, 101.9)
- moved SW3 3.80 mm to (167.1, 103.6)
- moved R12 3.67 mm to (122.3, 83.2), turned to -90 degrees
- moved C8 3.30 mm to (122.1, 76.2)
- moved R2 3.18 mm to (127.6, 119.7)
- moved R1 2.86 mm to (127.6, 116.8)
- moved J1 2.82 mm to (116.2, 110.0)
- moved R3 2.80 mm to (125.0, 110.2), turned to 0 degrees
- moved FB1 2.75 mm to (116.0, 90.9), turned to 0 degrees
- moved C4 1.98 mm to (184.7, 107.4)
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Connections:
- J3 pad A1: Net-(JP3-C) -> GND
- J3 pad A3: GND -> Net-(JP3-C)
- U3 pad 10: unconnected-(U3-GPIO25(DAC_1)-Pad10) -> Net-(U3-GPIO25(DAC_1))
- U3 pad 11: unconnected-(U3-GPIO26(DAC_2)-Pad11) -> Net-(U3-GPIO26(DAC_2))
Other:
- board text added: "MCU"
- board text added: "Power"
- board text added: "USB"
