File: ImogenWren.kicad_sch (KiCad schematic)
At the start: 3 parts

Commit message: dfghdreg
Parts:
- added BT1: Battery_Cell, symbol Device:Battery_Cell
- added C8: 100n, Capacitor_SMD:C_0805_2012Metric_Pad1.18x1.45mm_HandSolder, symbol 000_Capacitor_Film_Immo:cap_film_0805
- added R4: Resistor_0805, Resistor_SMD:R_0805_2012Metric_Pad1.20x1.40mm_HandSolder, symbol 000_Resistors_Immo:Resistor_0805
- added U3: MCP73831-2-OT, Package_TO_SOT_SMD:SOT-23-5, symbol Battery_Management:MCP73831-2-OT
Connections:
- net MCU/D+ is gone; now on net ESP32/D+: R3.1
- net MCU/D- is gone; now on net ESP32/D-: R2.1
- net USB/USB_POWER_OUT: now also U3.4 (V_{DD})
- new net BATTERY_POWER: BT1.1 (+), C8.1, U3.3 (V_{BAT})
- new net CHARGE_INHIBIT: R4.1, U3.5 (PROG)
- new net CHARGE_STATUS: U3.1 (STAT)
- new net GND: C8.2
- new net GNDPWR: BT1.2 (-), R4.2, U3.2 (V_{SS})
Other:
- removed sheet MCU
- sheet ESP32 ports: added LED_DATA_OUT; removed USB_PWR_OUT
- note added: "Programming Resistor Need multiple & jumpers?"
- moved on the sheet: D2, R2, R3

Commit message: dhdfbg
Other:
- added sheet Audio Driver (esp32-audio-output.kicad_sch)
- added sheet Buttons (buttons.kicad_sch)
- added sheet WS2812b LEDs (ws2812b-led-string.kicad_sch)
Changed lines of the file:
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@@
+    )
+  )
+  (sheet (at 90.17 147.32) (size 40.64 33.02) (fields_autoplaced)
+    (stroke (width 0.1524) (type solid))
+    (fill (color 0 0 0 0.0000))
+    (property "Sheetname" "Audio Driver" (at 90.17 146.6084 0)
+      (effects (font (size 1.27 1.27)) (justify left bottom))
+    )
+    (property "Sheetfile" "esp32-audio-output.kicad_sch" (at 90.17 180.9246 0)
+      (effects (font (size 1.27 1.27)) (justify left top))
+    )
+    (instances
+      (project "ImogenWren"
+        (path "/84b7ad53-68b5-40da-9777-f5bb9a09ecb4" (page "7"))
+      )
+    )
+  )
+  (sheet (at 222.25 45.72) (size 34.29 21.59) (fields_autoplaced)
+    (stroke (width 0.1524) (type solid))
+    (fill (color 0 0 0 0.0000))
+    (property "Sheetname" "WS2812b LEDs" (at 222.25 45.0084 0)
+      (effects (font (size 1.27 1.27)) (justify left bottom))
+    )
+    (property "Sheetfile" "ws2812b-led-string.kicad_sch" (at 222.25 67.8946 0)
+      (effects (font (size 1.27 1.27)) (justify left top))
+    )
+    (instances
+      (project "ImogenWren"
+        (path "/84b7ad53-68b5-40da-9777-f5bb9a09ecb4" (page "8"))
+      )
+    )
+  )
+  (sheet (at 168.91 121.92) (size 31.75 26.67) (fields_autoplaced)
+    (stroke (width 0.1524) (type solid))
+    (fill (color 0 0 0 0.0000))
+    (property "Sheetname" "Buttons" (at 168.91 121.2084 0)
+      (effects (font (size 1.27 1.27)) (justify left bottom))
+    )
+    (property "Sheetfile" "buttons.kicad_sch" (at 168.91 149.1746 0)
+      (effects (font (size 1.27 1.27)) (justify left top))
+    )
+    (instances
+      (project "ImogenWren"
+        (path "/84b7ad53-68b5-40da-9777-f5bb9a09ecb4" (page "6"))
+      )
     )
   )

Commit message: sdfdsfvsd
Parts:
- removed D2: PRTR5V0U2X, Package_TO_SOT_SMD:SOT-143, symbol Power_Protection:PRTR5V0U2X
- added EC1: 1000u, Capacitor_SMD:CP_Elec_10x10, symbol 000_Capacitor_Electrolytic_Immo:220u
- added JP1: Jumper_3_Bridged12, Jumper:SolderJumper-3_P1.3mm_Bridged12_RoundedPad1.0x1.5mm, symbol 000_Connectors_Immo:Jumper_3_Bridged12
- added JP2: I Prog, Jumper:SolderJumper-3_P1.3mm_Open_RoundedPad1.0x1.5mm_NumberLabels, symbol Jumper:SolderJumper_3_Open
- added R5: 10k, Resistor_SMD:R_0805_2012Metric_Pad1.20x1.40mm_HandSolder, symbol 000_Resistors_Immo:Resistor_0805
- added R6: 4k7, Resistor_SMD:R_0805_2012Metric_Pad1.20x1.40mm_HandSolder, symbol 000_Resistors_Immo:Resistor_0805
- added R7: 470r, Resistor_SMD:R_0805_2012Metric_Pad1.20x1.40mm_HandSolder, symbol 000_Resistors_Immo:Resistor_0805
- R4: value Resistor_0805 -> 10k
Connections:
- net BATTERY_POWER: now also JP1.1 (A); no longer C8.1
- net CHARGE_INHIBIT: now also R5.1, R6.1
- net ESP32/LED_DATA_OUT: now also R7.2
- net GND: now also EC1.2
- net GNDPWR: now also JP2.2 (C)
- new net: JP2.1 (A), R5.2
- new net: JP2.3 (B), R6.2
- new net ESP32/+5V_IN: C8.1, EC1.1, JP1.2 (C)
- new net USB_POWER: JP1.3 (B)
- new net WS2812b LEDs/DATA_IN: R7.1
Other:
- sheet WS2812b LEDs ports: added 5V_IN, DATA_IN, DATA_OUT, GND; removed none
- note added: "1 open, 3 open = 10 kohm = 100mA 1 close, 3 open = 4k7 ohm = ~ 250mA 1 open, 3 close = 3k1 ohm = ~ 350mA 1 close , 3 close = 2k4 ogm = ~ 500mA"
- note added: "Fast Charge Current Regulation IREG |Min. | Typ. | Max. | Units | Conditions | |90 |100 | 110 |mA |PROG = 10 kohm | |450 |505 | 550 |mA |PROG = 2.0 kohm| |12.5 | 14.5 | 16.5 |mA |PROG = 67 kohm | TA = -5°C to +55°C"
- moved on the sheet: R4

Commit message: n;kln;sfdg
Parts:
- added J8: WS2821_LED_OUT, Connector_Molex:Molex_KK-254_AE-6410-03A_1x03_P2.54mm_Vertical, symbol 000_Connectors_Immo:3pin_molex_2.54mm_male
- added JPw: Disable Onboard LEDs, Jumper:SolderJumper-2_P1.3mm_Bridged_RoundedPad1.0x1.5mm, symbol 000_Connectors_Immo:Jumper_2_Bridge_Small
Connections:
- net GND: now also J8.1 (Pin_1)
- net WS2812b LEDs/DATA_IN: now also J8.3 (Pin_3)
- net ESP32/+5V_IN renamed BATTERY_POWER_BUS
- net BATTERY_POWER_BUS: now also J8.2 (Pin_2), JPw.1 (A)
- new net WS2812b LEDs/5V_IN: JPw.2 (B)
Other:
- note added: "Can be much smaller"
- note added: "Careful power distribution! - Power Bus is Battery OR USB, or UNREGULATED Vin - Regulated to 3v3 for MCU - Do not apply >5v to Vin"
Changed lines of the file:
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@@
 (kicad_sch (version 20230121) (generator eeschema)
   (paper "A4")
+  (junction (at 199.39 55.88) (diameter 0) (color 0 0 0 0)
+  )
   (junction (at 123.19 49.53) (diameter 0) (color 0 0 0 0)
   )
@@
     (stroke (width 0) (type default))
   )
-  (wire (pts (xy 177.8 41.91) (xy 177.8 45.72))
+  (wire (pts (xy 181.61 41.91) (xy 181.61 45.72))
     (stroke (width 0) (type default))
   )
@@
     (stroke (width 0) (type default))
   )
-  (wire (pts (xy 181.61 41.91) (xy 177.8 41.91))
-    (stroke (width 0) (type default))
-  )
   (wire (pts (xy 181.61 31.75) (xy 181.61 33.02))
     (stroke (width 0) (type default))
   )
+  (wire (pts (xy 199.39 55.88) (xy 199.39 69.85))
+    (stroke (width 0) (type default))
+  )
   (wire (pts (xy 127 97.79) (xy 127 100.33))
     (stroke (width 0) (type default))
@@
     (stroke (width 0) (type default))
   )
+  (wire (pts (xy 199.39 69.85) (xy 243.84 69.85))
+    (stroke (width 0) (type default))
+  )
   (wire (pts (xy 87.63 44.45) (xy 109.22 44.45))
     (stroke (width 0) (type default))
@@
     (stroke (width 0) (type default))
   )
+  (wire (pts (xy 199.39 55.88) (xy 215.9 55.88))
+    (stroke (width 0) (type default))
+  )
+  (wire (pts (xy 190.5 72.39) (xy 243.84 72.39))
+    (stroke (width 0) (type default))
+  )
   (wire (pts (xy 91.44 81.28) (xy 91.44 92.71))
     (stroke (width 0) (type default))
@@
     (stroke (width 0) (type default))
   )
-  (wire (pts (xy 203.2 41.91) (xy 181.61 41.91))
+  (wire (pts (xy 204.47 31.75) (xy 215.9 31.75))
+    (stroke (width 0) (type default))
+  )
+  (wire (pts (xy 215.9 41.91) (xy 181.61 41.91))
     (stroke (width 0) (type default))
   )
@@
     (stroke (width 0) (type default))
   )
+  (wire (pts (xy 210.82 74.93) (xy 210.82 76.2))
+    (stroke (width 0) (type default))
+  )
   (wire (pts (xy 63.5 60.96) (xy 101.6 60.96))
     (stroke (width 0) (type default))
@@
     (stroke (width 0) (type default))
   )
-  (wire (pts (xy 195.58 55.88) (xy 203.2 55.88))
+  (wire (pts (xy 195.58 55.88) (xy 199.39 55.88))
     (stroke (width 0) (type default))
   )
@@
     (stroke (width 0) (type default))
   )
+  (wire (pts (xy 210.82 74.93) (xy 243.84 74.93))
+    (stroke (width 0) (type default))
+  )
   (wire (pts (xy 91.44 110.49) (xy 91.44 128.27))
     (stroke (width 0) (type default))
@@
     (stroke (width 0) (type default))
   )
-  (wire (pts (xy 181.61 31.75) (xy 203.2 31.75))
+  (wire (pts (xy 181.61 31.75) (xy 198.12 31.75))
     (stroke (width 0) (type default))
   )
@@
     (effects (font (size 1.27 1.27)) (justify left bottom))
   )
+  (text "Careful power distribution!\n - Power Bus is Battery OR USB, or UNREGULATED Vin\n - Regulated to 3v3 for MCU\n - Do not apply >5v to Vin"
+    (at 19.05 21.59 0)
+    (effects (font (size 1.27 1.27)) (justify left bottom))
+  )
+  (text "Can be much smaller" (at 181.61 40.64 0)
+    (effects (font (size 1.27 1.27)) (justify left bottom))
+  )
   (text "Battery" (at 82.55 25.4 0)
     (effects (font (size 1.27 1.27)) (justify left bottom))
@@
     (effects (font (size 1.27 1.27)) (justify right bottom))
   )
+  (label "BATTERY_POWER_BUS" (at 190.5 72.39 0) (fields_autoplaced)
+    (effects (font (size 1.27 1.27)) (justify left bottom))
+  )
+  (label "BATTERY_POWER_BUS" (at 142.24 31.75 0) (fields_autoplaced)
+    (effects (font (size 1.27 1.27)) (justify left bottom))
+  )
   (hierarchical_label "CHARGE_STATUS" (shape output) (at 104.14 102.87 0) (fields_autoplaced)
     (effects (font (size 1.27 1.27)) (justify left))
@@
   (hierarchical_label "CHARGE_INHIBIT" (shape input) (at 64.77 102.87 180) (fields_autoplaced)
     (effects (font (size 1.27 1.27)) (justify right))
+  )
+  (symbol (lib_id "000_Connectors_Immo:3pin_molex_2.54mm_male") (at 248.92 72.39 180) (unit 1)
+    (in_bom yes) (on_board yes) (dnp no) (fields_autoplaced)
+    (property "Reference" "J8" (at 250.19 71.755 0)
+      (effects (font (size 1.27 1.27)) (justify right))
+    )
+    (property "Value" "WS2821_LED_OUT" (at 250.19 74.295 0)
+      (effects (font (size 1.27 1.27)) (justify right))
+    )
+    (property "Footprint" "Connector_Molex:Molex_KK-254_AE-6410-03A_1x03_P2.54mm_Vertical" (at 245.491 65.405 0)
+      (effects (font (size 1.27 1.27)) hide)
+    )
+    (property "Datasheet" "~" (at 248.92 72.39 0)
+      (effects (font (size 1.27 1.27)) hide)
+    )
+    (pin "1")
+    (pin "2")
+    (pin "3")
+    (instances
+      (project "ImogenWren"
+        (path "/84b7ad53-68b5-40da-9777-f5bb9a09ecb4"
+          (reference "J8") (unit 1)
+        )
+      )
+    )
   )
   (symbol (lib_id "000_Capacitor_Electrolytic_Immo:220u") (at 181.61 36.83 0) (unit 1)
@@
     )
   )
-  (symbol (lib_id "power:GND") (at 177.8 45.72 0) (unit 1)
-    (in_bom yes) (on_board yes) (dnp no) (fields_autoplaced)
-    (property "Reference" "#PWR06" (at 177.8 52.07 0)
-      (effects (font (size 1.27 1.27)) hide)
-    )
-    (property "Value" "GND" (at 177.8 50.8 0)
-      (effects (font (size 1.27 1.27)))
-    )
-    (property "Footprint" "" (at 177.8 45.72 0)
-      (effects (font (size 1.27 1.27)) hide)
-    )
-    (property "Datasheet" "" (at 177.8 45.72 0)
+  (symbol (lib_id "power:GND") (at 181.61 45.72 0) (unit 1)
+    (in_bom yes) (on_board yes) (dnp no) (fields_autoplaced)
+    (property "Reference" "#PWR06" (at 181.61 52.07 0)
+      (effects (font (size 1.27 1.27)) hide)
+    )
+    (property "Value" "GND" (at 181.61 50.8 0)
+      (effects (font (size 1.27 1.27)))
+    )
+    (property "Footprint" "" (at 181.61 45.72 0)
+      (effects (font (size 1.27 1.27)) hide)
+    )
+    (property "Datasheet" "" (at 181.61 45.72 0)
       (effects (font (size 1.27 1.27)) hide)
     )
@@
         (path "/84b7ad53-68b5-40da-9777-f5bb9a09ecb4"
           (reference "#PWR06") (unit 1)
+        )
+      )
+    )
+  )
+  (symbol (lib_id "000_Connectors_Immo:Jumper_2_Bridge_Small") (at 201.295 31.75 0) (unit 1)
+    (in_bom yes) (on_board yes) (dnp no) (fields_autoplaced)
+    (property "Reference" "JPw" (at 201.2725 26.67 0)
+      (effects (font (size 1.27 1.27)))
+    )
+    (property "Value" "Disable Onboard LEDs" (at 201.2725 29.21 0)
+      (effects (font (size 1.27 1.27)))
+    )
+    (property "Footprint" "Jumper:SolderJumper-2_P1.3mm_Bridged_RoundedPad1.0x1.5mm" (at 201.93 37.465 0)
+      (effects (font (size 1.27 1.27)) hide)
+    )
+    (property "Datasheet" "~" (at 201.295 38.735 0)
+      (effects (font (size 1.27 1.27)) hide)
+    )
+    (pin "1")
+    (pin "2")
+    (instances
+      (project "ImogenWren"
+        (path "/84b7ad53-68b5-40da-9777-f5bb9a09ecb4"
+          (reference "JPw") (unit 1)
         )
       )
@@
         (path "/84b7ad53-68b5-40da-9777-f5bb9a09ecb4"
           (reference "R6") (unit 1)
+        )
+      )
+    )
+  )
+  (symbol (lib_id "power:GND") (at 210.82 76.2 0) (unit 1)
+    (in_bom yes) (on_board yes) (dnp no) (fields_autoplaced)
+    (property "Reference" "#PWR07" (at 210.82 82.55 0)
+      (effects (font (size 1.27 1.27)) hide)
+    )
+    (property "Value" "GND" (at 210.82 81.28 0)
+      (effects (font (size 1.27 1.27)))
+    )
+    (property "Footprint" "" (at 210.82 76.2 0)
+      (effects (font (size 1.27 1.27)) hide)
+    )
+    (property "Datasheet" "" (at 210.82 76.2 0)
+      (effects (font (size 1.27 1.27)) hide)
+    )
+    (pin "1")
+    (instances
+      (project "ImogenWren"
+        (path "/84b7ad53-68b5-40da-9777-f5bb9a09ecb4"
+          (reference "#PWR07") (unit 1)
         )
       )
@@
     )
   )
-  (sheet (at 203.2 29.21) (size 27.94 30.48) (fields_autoplaced)
+  (sheet (at 215.9 29.21) (size 27.94 30.48) (fields_autoplaced)
     (stroke (width 0.1524) (type solid))
     (fill (color 253 44 255 0.4400))
-    (property "Sheetname" "WS2812b LEDs" (at 203.2 28.4984 0)
+    (property "Sheetname" "WS2812b LEDs" (at 215.9 28.4984 0)
       (effects (font (size 1.27 1.27)) (justify left bottom))
     )
-    (property "Sheetfile" "ws2812b-led-string.kicad_sch" (at 203.2 60.2746 0)
+    (property "Sheetfile" "ws2812b-led-string.kicad_sch" (at 215.9 60.2746 0)
       (effects (font (size 1.27 1.27)) (justify left top))
     )
-    (pin "DATA_IN" input (at 203.2 55.88 180)
-      (effects (font (size 1.27 1.27)) (justify left))
-    )
-    (pin "DATA_OUT" output (at 231.14 55.88 0)
+    (pin "DATA_IN" input (at 215.9 55.88 180)
+      (effects (font (size 1.27 1.27)) (justify left))
+    )
+    (pin "DATA_OUT" output (at 243.84 55.88 0)
       (effects (font (size 1.27 1.27)) (justify right))
     )
-    (pin "5V_IN" input (at 203.2 31.75 180)
-      (effects (font (size 1.27 1.27)) (justify left))
-    )
-    (pin "GND" passive (at 203.2 41.91 180)
-      (effects (font (size 1.27 1.27)) (justify left))
-    )
+    (pin "5V_IN" input (at 215.9 31.75 180)
+      (effects (font (size 1.27 1.27)) (justify left))
+    )
+    (pin "GND" passive (at 215.9 41.91 180)
+      (effects (font (size 1.27 1.27)) (justify left))
+    )

Commit message: werewr
Parts:
- added JP3: LED_DATA_SOURCE, Jumper:SolderJumper-3_P1.3mm_Bridged12_RoundedPad1.0x1.5mm, symbol 000_Connectors_Immo:Jumper_3_Bridged12
Connections:
- net WS2812b LEDs/DATA_IN: now also JP3.1 (A); no longer J8.3 (Pin_3)
- net WS2812b LEDs/DATA_OUT: now also JP3.3 (B)
- new net: J8.3 (Pin_3), JP3.2 (C)
Other:
- moved on the sheet: J8
Changed lines of the file:
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@@
+    (stroke (width 0) (type default))
+  )
+  (wire (pts (xy 252.73 55.88) (xy 243.84 55.88))
     (stroke (width 0) (type default))
   )
@@
     (stroke (width 0) (type default))
   )
-  (wire (pts (xy 199.39 55.88) (xy 199.39 69.85))
+  (wire (pts (xy 199.39 55.88) (xy 199.39 73.66))
     (stroke (width 0) (type default))
   )
@@
     (stroke (width 0) (type default))
   )
-  (wire (pts (xy 199.39 69.85) (xy 243.84 69.85))
+  (wire (pts (xy 199.39 73.66) (xy 226.06 73.66))
+    (stroke (width 0) (type default))
+  )
+  (wire (pts (xy 252.73 73.66) (xy 252.73 55.88))
     (stroke (width 0) (type default))
   )
@@
     (stroke (width 0) (type default))
   )
-  (wire (pts (xy 190.5 72.39) (xy 243.84 72.39))
+  (wire (pts (xy 190.5 80.01) (xy 243.84 80.01))
     (stroke (width 0) (type default))
   )
@@
     (stroke (width 0) (type default))
   )
-  (wire (pts (xy 210.82 74.93) (xy 210.82 76.2))
+  (wire (pts (xy 210.82 82.55) (xy 210.82 83.82))
     (stroke (width 0) (type default))
   )
@@
     (stroke (width 0) (type default))
   )
-  (wire (pts (xy 210.82 74.93) (xy 243.84 74.93))
+  (wire (pts (xy 210.82 82.55) (xy 243.84 82.55))
     (stroke (width 0) (type default))
   )
@@
     (stroke (width 0) (type default))
   )
+  (wire (pts (xy 233.68 73.66) (xy 252.73 73.66))
+    (stroke (width 0) (type default))
+  )
   (wire (pts (xy 63.5 81.28) (xy 91.44 81.28))
     (stroke (width 0) (type default))
@@
   )
   (wire (pts (xy 68.58 121.92) (xy 68.58 134.62))
+    (stroke (width 0) (type default))
+  )
+  (wire (pts (xy 229.87 77.47) (xy 243.84 77.47))
     (stroke (width 0) (type default))
   )
@@
     (effects (font (size 1.27 1.27)) (justify right bottom))
   )
-  (label "BATTERY_POWER_BUS" (at 190.5 72.39 0) (fields_autoplaced)
+  (label "BATTERY_POWER_BUS" (at 190.5 80.01 0) (fields_autoplaced)
     (effects (font (size 1.27 1.27)) (justify left bottom))
   )
@@
     (effects (font (size 1.27 1.27)) (justify right))
   )
-  (symbol (lib_id "000_Connectors_Immo:3pin_molex_2.54mm_male") (at 248.92 72.39 180) (unit 1)
-    (in_bom yes) (on_board yes) (dnp no) (fields_autoplaced)
-    (property "Reference" "J8" (at 250.19 71.755 0)
+  (symbol (lib_id "000_Connectors_Immo:3pin_molex_2.54mm_male") (at 248.92 80.01 180) (unit 1)
+    (in_bom yes) (on_board yes) (dnp no) (fields_autoplaced)
+    (property "Reference" "J8" (at 250.19 79.375 0)
       (effects (font (size 1.27 1.27)) (justify right))
     )
-    (property "Value" "WS2821_LED_OUT" (at 250.19 74.295 0)
+    (property "Value" "WS2821_LED_OUT" (at 250.19 81.915 0)
       (effects (font (size 1.27 1.27)) (justify right))
     )
-    (property "Footprint" "Connector_Molex:Molex_KK-254_AE-6410-03A_1x03_P2.54mm_Vertical" (at 245.491 65.405 0)
-      (effects (font (size 1.27 1.27)) hide)
-    )
-    (property "Datasheet" "~" (at 248.92 72.39 0)
+    (property "Footprint" "Connector_Molex:Molex_KK-254_AE-6410-03A_1x03_P2.54mm_Vertical" (at 245.491 73.025 0)
+      (effects (font (size 1.27 1.27)) hide)
+    )
+    (property "Datasheet" "~" (at 248.92 80.01 0)
       (effects (font (size 1.27 1.27)) hide)
     )
@@
     )
   )
+  (symbol (lib_id "000_Connectors_Immo:Jumper_3_Bridged12") (at 229.87 73.66 0) (unit 1)
+    (in_bom yes) (on_board yes) (dnp no) (fields_autoplaced)
+    (property "Reference" "JP3" (at 229.87 69.85 0)
+      (effects (font (size 1.27 1.27)))
+    )
+    (property "Value" "LED_DATA_SOURCE" (at 229.87 72.39 0)
+      (effects (font (size 1.27 1.27)))
+    )
+    (property "Footprint" "Jumper:SolderJumper-3_P1.3mm_Bridged12_RoundedPad1.0x1.5mm" (at 230.505 84.328 0)
+      (effects (font (size 1.27 1.27)) hide)
+    )
+    (property "Datasheet" "~" (at 235.458 77.089 0)
+      (effects (font (size 1.27 1.27)) hide)
+    )
+    (pin "1")
+    (pin "2")
+    (pin "3")
+    (instances
+      (project "ImogenWren"
+        (path "/84b7ad53-68b5-40da-9777-f5bb9a09ecb4"
+          (reference "JP3") (unit 1)
+        )
+      )
+    )
+  )
   (symbol (lib_id "000_Resistors_Immo:Resistor_0805") (at 74.93 110.49 0) (unit 1)
     (in_bom yes) (on_board yes) (dnp no) (fields_autoplaced)
@@
     )
   )
-  (symbol (lib_id "power:GND") (at 210.82 76.2 0) (unit 1)
-    (in_bom yes) (on_board yes) (dnp no) (fields_autoplaced)
-    (property "Reference" "#PWR07" (at 210.82 82.55 0)
-      (effects (font (size 1.27 1.27)) hide)
-    )
-    (property "Value" "GND" (at 210.82 81.28 0)
-      (effects (font (size 1.27 1.27)))
-    )
-    (property "Footprint" "" (at 210.82 76.2 0)
-      (effects (font (size 1.27 1.27)) hide)
-    )
-    (property "Datasheet" "" (at 210.82 76.2 0)
-      (effects (font (size 1.27 1.27)) hide)
-    )
+  (symbol (lib_id "power:GND") (at 210.82 83.82 0) (unit 1)
+    (in_bom yes) (on_board yes) (dnp no) (fields_autoplaced)
+    (property "Reference" "#PWR07" (at 210.82 90.17 0)
+      (effects (font (size 1.27 1.27)) hide)
+    )
+    (property "Value" "GND" (at 210.82 88.9 0)
+      (effects (font (size 1.27 1.27)))
+    )
+    (property "Footprint" "" (at 210.82 83.82 0)
+      (effects (font (size 1.27 1.27)) hide)
+    )
+    (property "Datasheet" "" (at 210.82 83.82 0)
+      (effects (font (size 1.27 1.27)) hide)
+    )

Commit message: kjsaofklihsdof
Parts:
- removed R2, R3: 27r, Resistor_SMD:R_0805_2012Metric_Pad1.20x1.40mm_HandSolder, symbol 000_Resistors_Immo:Resistor_0805
- added R4, R5: 27r, Resistor_SMD:R_0805_2012Metric_Pad1.20x1.40mm_HandSolder, symbol 000_Resistors_Immo:Resistor_0805
- added SW1: Power, Button_Switch_SMD:SW_SPDT_PCM12, symbol Switch:SW_SPST
- BT1: footprint (none) -> Battery:BatteryHolder_Keystone_1060_1x2032
- J1: renamed from J8; footprint Connector_Molex:Molex_KK-254_AE-6410-03A_1x03_P2.54mm_Vertical -> Connector_PCBEdge:BUS_PCIexpress_x1
- JP2: renamed from JP1; value Jumper_3_Bridged12 -> Power Routing
- renumbered C8 to C1, JP2 to JP1, JPw to JPw1, R4 to R1, R5 to R2, R6 to R3, R7 to R6, U3 to U1
Connections:
- net USB/USB_POWER_OUT is gone; now on net USB_POWER: U1.4 (V_{DD})
- net BATTERY_POWER: now also SW1.1 (A); no longer BT1.1 (+)
- net ESP32/D+: now also R5.1
- net ESP32/D-: now also R4.1
- net USB/D+: now also R5.2
- net USB/D-: now also R4.2
- new net: BT1.1 (+), SW1.2 (B)
Other:
- moved on the sheet: BT1

Commit message: xcfgdfgd
Parts:
- removed BT1: Battery_Cell, Battery:BatteryHolder_Keystone_1060_1x2032, symbol Device:Battery_Cell
- removed J1: WS2821_LED_OUT, Connector_PCBEdge:BUS_PCIexpress_x1, symbol 000_Connectors_Immo:3pin_molex_2.54mm_male
- removed SW1: Power, Button_Switch_SMD:SW_SPDT_PCM12, symbol Switch:SW_SPST
- added J1: Battery Cell 4.2v, 000-edge-connectors-immo:2-pin-edge, symbol 000-lost-edge-connectors:2-pin-edge-touch
- added J3: WS2821b-LED-Out, 000-edge-connectors-immo:3-pin-edge, symbol 000-lost-edge-connectors:3-pin-edge-touch
- added SW1: SW_SPDT_small, 000_Switches_Immo:SW_SPDT_PCM12, symbol 000_Switches_Immo:SW_SPDT_small
Connections:
- net BATTERY_POWER: now also SW1.1 (A)
- net BATTERY_POWER_BUS: now also J3.A2
- net GND: now also J3.A3
- net GNDPWR: now also J1.A1
- net at JP3.2 (C): now also J3.A1
- new net: J1.A2, SW1.2 (B)
