File: ImogenWren.kicad_sch (KiCad schematic)
At the start: 16 parts, among them J1 Battery Cell 4.2v, J3 WS2821b-LED-Out, SW1 SW_SPDT_small, U1 MCP73831-2-OT

Commit message: desgfdfg
Parts:
- J1: symbol 000-lost-edge-connectors:2-pin-edge-touch -> 000-edge-connectors-immo:2-pin-edge-touch; PIN1 gnd -> Batt-; PIN2 Batt_4.2v -> Batt+
- J3: symbol 000-lost-edge-connectors:3-pin-edge-touch -> 000-edge-connectors-immo:3-pin-edge-touch
Other:
- note added: "Change jumper if omitting battery"
Changed lines of the file:
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@@
+    (effects (font (size 1.27 1.27)) (justify left bottom))
+  )
+  (text "Change jumper if omitting battery" (at 86.36 28.575 0)
     (effects (font (size 1.27 1.27)) (justify left bottom))
   )
@@
     )
   )
-  (symbol (lib_id "000-lost-edge-connectors:3-pin-edge-touch") (at 259.08 92.71 0) (unit 1)
+  (symbol (lib_id "000-edge-connectors-immo:3-pin-edge-touch") (at 259.08 92.71 0) (unit 1)
     (in_bom yes) (on_board yes) (dnp no)
     (property "Reference" "J3" (at 255.905 72.39 0)
@@
       (effects (font (size 1.27 1.27)) hide)
     )
-    (property "PIN1_NAME" "D" (at 266.7 78.74 0)
-      (effects (font (size 1.27 1.27)))
-    )
-    (property "PIN2_NAME" "V+" (at 266.065 80.645 0)
-      (effects (font (size 1.27 1.27)))
-    )
-    (property "PIN3_NAME" "G" (at 266.7 82.55 0)
+    (property "PIN1_NAME" "D" (at 265.43 78.74 0)
+      (effects (font (size 1.27 1.27)))
+    )
+    (property "PIN2_NAME" "V+" (at 266.7 81.28 0)
+      (effects (font (size 1.27 1.27)))
+    )
+    (property "PIN3_NAME" "G" (at 265.43 82.55 0)
       (effects (font (size 1.27 1.27)))
     )
@@
     )
   )
-  (symbol (lib_id "000-lost-edge-connectors:2-pin-edge-touch") (at 141.605 107.315 0) (mirror x) (unit 1)
+  (symbol (lib_id "000-edge-connectors-immo:2-pin-edge-touch") (at 141.605 107.315 0) (mirror x) (unit 1)
     (in_bom yes) (on_board yes) (dnp no)
     (property "Reference" "J1" (at 132.08 100.33 0)
@@
       (effects (font (size 1.27 1.27)) hide)
     )
-    (property "PIN1" "gnd" (at 149.86 107.315 0)
-      (effects (font (size 1.27 1.27)) (justify left))
-    )
-    (property "PIN2" "Batt_4.2v" (at 149.86 105.41 0)
-      (effects (font (size 1.27 1.27)) (justify left))
+    (property "PIN1" "Batt-" (at 152.4 107.95 0)
+      (effects (font (size 1.27 1.27)))
+    )
+    (property "PIN2" "Batt+" (at 152.4 105.41 0)
+      (effects (font (size 1.27 1.27)))
     )
     (pin "A1")
