File: ISOpower_ESP32.kicad_sch (KiCad schematic)
At the start: 15 parts, among them J2 ESP_GPIO_B, J3 ESPpin4-7, J4 SDI-SDO, J5 ESP_GPIO_A, J7 i2c Header, U1 ESP32-WROOM-32, U2 AMS1117-3.3

Commit message: dfghdreg
Parts:
- removed J5: ESP_GPIO_A, Connector_PinHeader_1.27mm:PinHeader_1x10_P1.27mm_Vertical, symbol Connector:Conn_01x10_Male
- added J6: Conn_01x10_Pin, Connector_PinHeader_2.00mm:PinHeader_1x10_P2.00mm_Vertical, symbol 000_Pin_Headers_Immo:Conn_01x10_Pin
Connections:
- net at U1.8 (GPIO32): now also J6.1 (Pin_1)
- net at D9.2 (A), U1.24 (GPIO2): now also J6.10 (Pin_10)
- net at U1.9 (GPIO33): now also J6.2 (Pin_2)
- net at U1.10 (GPIO25): now also J6.3 (Pin_3)
- net at U1.11 (GPIO26): now also J6.4 (Pin_4)
- net at U1.12 (GPIO27): now also J6.5 (Pin_5)
- net at U1.13 (GPIO14): now also J6.6 (Pin_6)
- net at U1.14 (GPIO12): now also J6.7 (Pin_7)
- net at U1.16 (GPIO13): now also J6.8 (Pin_8)
- net at U1.23 (GPIO15): now also J6.9 (Pin_9)
- net 5: no longer names the net of J2.4 (Pin_4)
- net 5: no longer U1.29 (GPIO5)
- new net LED_DATA_OUT: U1.29 (GPIO5)

Commit message: n;kln;sfdg
Parts:
- removed J7: i2c Header, Connector_PinHeader_1.27mm:PinHeader_1x05_P1.27mm_Vertical, symbol Connector:Conn_01x05_Male
- added J5: i2c Header, Connector_PinHeader_1.27mm:PinHeader_1x05_P1.27mm_Vertical, symbol Connector:Conn_01x05_Male
- added J7: Bus_PCI_Express_x1, symbol Connector:Bus_PCI_Express_x1
- J6: value Conn_01x10_Pin -> ESP_GPIO_A [Make New Part & Label
Connections:
- net Logic Level Conversion/0A is gone; now on net SSERIAL_RX: U1.28 (UART2_TX/GPIO17)
- net Logic Level Conversion/1A is gone; now on net SSERIAL_TX: U1.27 (UART2_RX/GPIO16)
- net +5V_IN: now also J5.5 (Pin_5)
- net 3V3_OUT: now also J5.4 (Pin_4)
- net GND: now also J5.1 (Pin_1)
- net SCL: now also J5.2 (Pin_2)
- net SDA: now also J5.3 (Pin_3)
- net GPIO32: now reaches J6.1 (Pin_1), U1.8 (GPIO32)
- new net: J7.A10 (+3.3V), J7.A9 (+3.3V), J7.B8 (+3.3V)
- new net: J7.A12 (GND), J7.A15 (GND), J7.A18 (GND), J7.A4 (GND), J7.B13 (GND), J7.B16 (GND), J7.B18 (GND), J7.B4 (GND), J7.B7 (GND)
- new net: J7.A2 (+12V), J7.A3 (+12V), J7.B1 (+12V), J7.B2 (+12V), J7.B3 (+12V)
Other:
- removed sheet Logic Level Conversion
- moved on the sheet: R2, R3

Commit message: werewr
Parts:
- removed J4: SDI-SDO, Connector_PinHeader_1.27mm:PinHeader_1x06_P1.27mm_Vertical, symbol Connector:Conn_01x06_Male
- removed J6: ESP_GPIO_A [Make New Part & Label, Connector_PinHeader_2.00mm:PinHeader_1x10_P2.00mm_Vertical, symbol 000_Pin_Headers_Immo:Conn_01x10_Pin
- removed J7: Bus_PCI_Express_x1, symbol Connector:Bus_PCI_Express_x1
- removed U1: ESP32-WROOM-32, RF_Module:ESP32-WROOM-32, symbol 000_MCU_microcontrollers_Immo:ESP32-WROOM-32
- added J4: 1-pin-edge-touch-XL, Connector_PCBEdge:BUS_PCIexpress_x1, symbol 000-edge-connectors-immo:1-pin-edge-touch-XL
- added J6: Touch Pins, Connector_PCBEdge:BUS_PCIexpress_x1, symbol 000-edge-connectors-immo:8-pin-edge-touch
- added J7: SDI/SDO, Connector_PCBEdge:BUS_PCIexpress_x1, symbol 000-edge-connectors-immo:6-pin-edge-touch
- added U4: ESP32-WROOM-32, RF_Module:ESP32-WROOM-32, symbol 000_MCU_microcontrollers_Immo:ESP32-WROOM-32_2
Connections:
- net 19: now also U4.31 (GPIO19)
- net 3V3_OUT: now also U4.2 (VDD)
- net GND: now also U4.1 (GND), U4.15 (GND), U4.38 (GND), U4.39 (GND)
- net LED_DATA_OUT: now also U4.29 (GPIO5)
- net SCL: now also U4.36 (GPIO22)
- net SDA: now also U4.33 (GPIO21)
- net SSERIAL_RX: now also U4.28 (UART2_TX/GPIO17)
- net SSERIAL_TX: now also U4.27 (UART2_RX/GPIO16)
- net USB ESP32 CH340 Interface /ESP_EN: now also U4.3 (EN)
- net USB ESP32 CH340 Interface /ESP_IO0: now also U4.25 (IO0/GPIO0/T1)
- net USB ESP32 CH340 Interface /RxD_B: now also U4.35 (TXD0/GPIO1)
- net USB ESP32 CH340 Interface /TxD_B: now also U4.34 (RXD0/GPIO3)
- net at D9.2 (A): now also U4.37 (GPIO23)
- net at J3.1 (Pin_1): now also U4.4 (SENSOR_VP)
- net at J3.2 (Pin_2): now also U4.5 (SENSOR_VN)
- net at J3.3 (Pin_3): now also U4.6 (IO34)
- net at J3.4 (Pin_4): now also U4.7 (IO35)
- new net: J4.A1, U4.26 (GPIO4(T0))
- new net: J6.A6, U4.12 (GPIO27(T7))
- new net: J6.A5, U4.13 (GPIO14(T6))
- new net: J6.A4, U4.14 (GPIO12(T5))
- new net: J6.A3, U4.16 (GPIO13(T4))
- new net: J7.A6, U4.17 (SHD/SD2)
- new net: J7.A5, U4.18 (SWP/SD3)
- new net: J7.A4, U4.19 (SCS/CMD)
- new net: J7.A3, U4.20 (SCK/CLK)
- new net: J7.A2, U4.21 (SDO/SD0)
- new net: J7.A1, U4.22 (SDI/SD1)
- new net: J6.A2, U4.23 (GPIO15(T3))
- new net: J6.A1, U4.24 (GPIO2(T2))
- new net: J6.A8, U4.8 (GPIO32(T9))
- new net: J6.A7, U4.9 (GPIO33(T8))
Other:
- moved on the sheet: D9, R30

Commit message: kjsaofklihsdof
Parts:
- J3: renamed from J2; footprint Connector_PinHeader_1.27mm:PinHeader_1x05_P1.27mm_Vertical -> Connector_PCBEdge:BUS_PCIexpress_x1
- J4: renamed from J3; footprint Connector_PinHeader_1.27mm:PinHeader_1x04_P1.27mm_Vertical -> Connector_PCBEdge:BUS_PCIexpress_x1
- J6: footprint Connector_PCBEdge:BUS_PCIexpress_x1 -> 000-edge-connectors-immo:8-pin-edge-touch
- J7: renamed from J5; footprint Connector_PinHeader_1.27mm:PinHeader_1x05_P1.27mm_Vertical -> Connector_PCBEdge:BUS_PCIexpress_x1
- renumbered C5 to C3, C1 to C4, C3 to C5, D9 to D1, J7 to J2, J4 to J5, R30 to R7, R3 to R8, R2 to R9, U4 to U3
Changed lines of the file:
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@@
   (symbol (lib_id "000-edge-connectors-immo:1-pin-edge-touch-XL") (at 200.66 115.57 0) (unit 1)
     (in_bom yes) (on_board yes) (dnp no) (fields_autoplaced)
-    (property "Reference" "J4" (at 207.01 101.6 0)
+    (property "Reference" "J5" (at 207.01 101.6 0)
       (effects (font (size 1.27 1.27)) (justify left))
     )
@@
       (project "ImogenWren"
         (path "/84b7ad53-68b5-40da-9777-f5bb9a09ecb4/9cdb06a8-babb-4d9b-a75e-e6e2cfc518a0"
-          (reference "J4") (unit 1)
+          (reference "J5") (unit 1)
         )
       )
@@
   (symbol (lib_id "000_MCU_microcontrollers_Immo:ESP32-WROOM-32_2") (at 140.97 106.68 0) (unit 1)
     (in_bom yes) (on_board yes) (dnp no) (fields_autoplaced)
-    (property "Reference" "U4" (at 139.1159 69.85 0)
+    (property "Reference" "U3" (at 139.1159 69.85 0)
       (effects (font (size 1.27 1.27)) (justify left))
     )
@@
       (project "ImogenWren"
         (path "/84b7ad53-68b5-40da-9777-f5bb9a09ecb4/9cdb06a8-babb-4d9b-a75e-e6e2cfc518a0"
-          (reference "U4") (unit 1)
+          (reference "U3") (unit 1)
         )
       )
@@
   (symbol (lib_id "000_Resistors_Immo:Resistor_0805") (at 248.92 151.13 0) (unit 1)
     (in_bom yes) (on_board yes) (dnp no)
-    (property "Reference" "R2" (at 243.84 149.86 0)
+    (property "Reference" "R9" (at 243.84 149.86 0)
       (effects (font (size 1.27 1.27)) (justify left))
     )
@@
       (project "ImogenWren"
         (path "/84b7ad53-68b5-40da-9777-f5bb9a09ecb4/9cdb06a8-babb-4d9b-a75e-e6e2cfc518a0"
-          (reference "R2") (unit 1)
+          (reference "R9") (unit 1)
         )
       )
@@
       (effects (font (size 1.27 1.27)) (justify left))
     )
-    (property "Footprint" "Connector_PCBEdge:BUS_PCIexpress_x1" (at 215.9 166.37 0)
+    (property "Footprint" "000-edge-connectors-immo:8-pin-edge-touch" (at 215.9 166.37 0)
       (effects (font (size 1.27 1.27)) hide)
     )
@@
   (symbol (lib_id "Connector:Conn_01x05_Male") (at 105.41 148.59 0) (unit 1)
     (in_bom yes) (on_board yes) (dnp no) (fields_autoplaced)
-    (property "Reference" "J2" (at 106.045 138.43 0)
+    (property "Reference" "J3" (at 106.045 138.43 0)
       (effects (font (size 1.27 1.27)))
     )
@@
       (effects (font (size 1.27 1.27)))
     )
-    (property "Footprint" "Connector_PinHeader_1.27mm:PinHeader_1x05_P1.27mm_Vertical" (at 105.41 148.59 0)
+    (property "Footprint" "Connector_PCBEdge:BUS_PCIexpress_x1" (at 105.41 148.59 0)
       (effects (font (size 1.27 1.27)) hide)
     )
@@
       (project "ImogenWren"
         (path "/84b7ad53-68b5-40da-9777-f5bb9a09ecb4/9cdb06a8-babb-4d9b-a75e-e6e2cfc518a0"
-          (reference "J2") (unit 1)
+          (reference "J3") (unit 1)
         )
       )
@@
   (symbol (lib_id "power:PWR_FLAG") (at 48.26 29.21 180) (unit 1)
     (in_bom yes) (on_board yes) (dnp no) (fields_autoplaced)
-    (property "Reference" "#FLG0101" (at 48.26 31.115 0)
+    (property "Reference" "#FLG01" (at 48.26 31.115 0)
       (effects (font (size 1.27 1.27)) hide)
     )
@@
       (project "ImogenWren"
         (path "/84b7ad53-68b5-40da-9777-f5bb9a09ecb4/9cdb06a8-babb-4d9b-a75e-e6e2cfc518a0"
-          (reference "#FLG0101") (unit 1)
+          (reference "#FLG01") (unit 1)
         )
       )
@@
   (symbol (lib_id "000_Resistors_Immo:Resistor_0805") (at 166.37 63.5 90) (unit 1)
     (in_bom yes) (on_board yes) (dnp no)
-    (property "Reference" "R30" (at 165.0999 60.96 0)
+    (property "Reference" "R7" (at 165.0999 60.96 0)
       (effects (font (size 1.27 1.27)) (justify left))
     )
@@
       (project "ImogenWren"
         (path "/84b7ad53-68b5-40da-9777-f5bb9a09ecb4/9cdb06a8-babb-4d9b-a75e-e6e2cfc518a0"
-          (reference "R30") (unit 1)
+          (reference "R7") (unit 1)
         )
       )
@@
   (symbol (lib_id "000_Diodes_Immo:LED_0805_smd") (at 157.48 63.5 180) (unit 1)
     (in_bom yes) (on_board yes) (dnp no)
-    (property "Reference" "D9" (at 158.75 59.69 0)
+    (property "Reference" "D1" (at 158.75 59.69 0)
       (effects (font (size 1.27 1.27)) (justify right))
     )
@@
       (project "ImogenWren"
         (path "/84b7ad53-68b5-40da-9777-f5bb9a09ecb4/9cdb06a8-babb-4d9b-a75e-e6e2cfc518a0"
-          (reference "D9") (unit 1)
+          (reference "D1") (unit 1)
         )
       )
@@
   (symbol (lib_id "000-edge-connectors-immo:6-pin-edge-touch") (at 100.33 118.11 0) (mirror y) (unit 1)
     (in_bom yes) (on_board yes) (dnp no) (fields_autoplaced)
-    (property "Reference" "J7" (at 103.505 96.52 0)
+    (property "Reference" "J2" (at 103.505 96.52 0)
       (effects (font (size 1.27 1.27)))
     )
@@
       (project "ImogenWren"
         (path "/84b7ad53-68b5-40da-9777-f5bb9a09ecb4/9cdb06a8-babb-4d9b-a75e-e6e2cfc518a0"
-          (reference "J7") (unit 1)
+          (reference "J2") (unit 1)
         )
       )
@@
   (symbol (lib_id "Connector:Conn_01x05_Male") (at 271.78 156.21 180) (unit 1)
     (in_bom yes) (on_board yes) (dnp no)
-    (property "Reference" "J5" (at 273.05 157.4801 0)
+    (property "Reference" "J7" (at 273.05 157.4801 0)
       (effects (font (size 1.27 1.27)) (justify right))
     )
@@
       (effects (font (size 1.27 1.27)) (justify right))
     )
-    (property "Footprint" "Connector_PinHeader_1.27mm:PinHeader_1x05_P1.27mm_Vertical" (at 271.78 156.21 0)
+    (property "Footprint" "Connector_PCBEdge:BUS_PCIexpress_x1" (at 271.78 156.21 0)
       (effects (font (size 1.27 1.27)) hide)
     )
@@
       (project "ImogenWren"
         (path "/84b7ad53-68b5-40da-9777-f5bb9a09ecb4/9cdb06a8-babb-4d9b-a75e-e6e2cfc518a0"
-          (reference "J5") (unit 1)
+          (reference "J7") (unit 1)
         )
       )
@@
   (symbol (lib_id "000_Capacitor_Film_Immo:cap_film_0805") (at 83.82 35.56 0) (unit 1)
     (in_bom yes) (on_board yes) (dnp no) (fields_autoplaced)
-    (property "Reference" "C5" (at 87.63 34.2899 0)
+    (property "Reference" "C3" (at 87.63 34.2899 0)
       (effects (font (size 1.27 1.27)) (justify left))
     )
@@
       (project "ImogenWren"
         (path "/84b7ad53-68b5-40da-9777-f5bb9a09ecb4/9cdb06a8-babb-4d9b-a75e-e6e2cfc518a0"
-          (reference "C5") (unit 1)
+          (reference "C3") (unit 1)
         )
       )
@@
   (symbol (lib_id "000_Capacitor_Film_Immo:cap_film_0805") (at 116.84 59.69 0) (unit 1)
     (in_bom yes) (on_board yes) (dnp no)
-    (property "Reference" "C1" (at 118.11 57.15 0)
+    (property "Reference" "C4" (at 118.11 57.15 0)
       (effects (font (size 1.27 1.27)) (justify left))
     )
@@
       (project "ImogenWren"
         (path "/84b7ad53-68b5-40da-9777-f5bb9a09ecb4/9cdb06a8-babb-4d9b-a75e-e6e2cfc518a0"
-          (reference "C1") (unit 1)
+          (reference "C4") (unit 1)
         )
       )
@@
   (symbol (lib_id "Connector:Conn_01x04_Male") (at 110.49 83.82 0) (unit 1)
     (in_bom yes) (on_board yes) (dnp no) (fields_autoplaced)
-    (property "Reference" "J3" (at 111.125 76.2 0)
+    (property "Reference" "J4" (at 111.125 76.2 0)
       (effects (font (size 1.27 1.27)))
     )
@@
       (effects (font (size 1.27 1.27)))
     )
-    (property "Footprint" "Connector_PinHeader_1.27mm:PinHeader_1x04_P1.27mm_Vertical" (at 110.49 83.82 0)
+    (property "Footprint" "Connector_PCBEdge:BUS_PCIexpress_x1" (at 110.49 83.82 0)
       (effects (font (size 1.27 1.27)) hide)
     )
@@
       (project "ImogenWren"
         (path "/84b7ad53-68b5-40da-9777-f5bb9a09ecb4/9cdb06a8-babb-4d9b-a75e-e6e2cfc518a0"
-          (reference "J3") (unit 1)
+          (reference "J4") (unit 1)
         )
       )
@@
   (symbol (lib_id "000_Resistors_Immo:Resistor_0805") (at 231.14 151.13 0) (unit 1)
     (in_bom yes) (on_board yes) (dnp no)
-    (property "Reference" "R3" (at 227.33 149.86 0)
+    (property "Reference" "R8" (at 227.33 149.86 0)
       (effects (font (size 1.27 1.27)) (justify left))
     )
@@
       (project "ImogenWren"
         (path "/84b7ad53-68b5-40da-9777-f5bb9a09ecb4/9cdb06a8-babb-4d9b-a75e-e6e2cfc518a0"
-          (reference "R3") (unit 1)
+          (reference "R8") (unit 1)
         )
       )
@@
   (symbol (lib_id "000_Capacitor_Film_Immo:cap_film_0805") (at 125.73 59.69 0) (unit 1)
     (in_bom yes) (on_board yes) (dnp no)
-    (property "Reference" "C3" (at 127 57.15 0)
+    (property "Reference" "C5" (at 127 57.15 0)
       (effects (font (size 1.27 1.27)))
     )
@@
       (project "ImogenWren"
         (path "/84b7ad53-68b5-40da-9777-f5bb9a09ecb4/9cdb06a8-babb-4d9b-a75e-e6e2cfc518a0"
-          (reference "C3") (unit 1)
-        )
-      )
+          (reference "C5") (unit 1)
+        )
+      )

Commit message: ;j;lkjh;k
Parts:
- J5: footprint Connector_PCBEdge:BUS_PCIexpress_x1 -> 000-edge-connectors-immo:1-pin-edge-touch-xl
Changed lines of the file:
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@@
       (effects (font (size 1.27 1.27)) (justify left))
     )
-    (property "Footprint" "Connector_PCBEdge:BUS_PCIexpress_x1" (at 215.9 154.94 0)
+    (property "Footprint" "000-edge-connectors-immo:1-pin-edge-touch-xl" (at 215.9 154.94 0)
       (effects (font (size 1.27 1.27)) hide)
     )

Commit message: xcfgdfgd
Parts:
- removed J3: ESP_GPIO_B, Connector_PCBEdge:BUS_PCIexpress_x1, symbol Connector:Conn_01x05_Male
- removed J4: ESPpin4-7, Connector_PCBEdge:BUS_PCIexpress_x1, symbol Connector:Conn_01x04_Male
- removed J7: i2c Header, Connector_PCBEdge:BUS_PCIexpress_x1, symbol Connector:Conn_01x05_Male
- added J10: ESPpin1-4, 000-edge-connectors-immo:4-pin-edge, symbol 000-lost-edge-connectors:4-pin-edge-touch
- added J4: ESP-gpio-B, 000-edge-connectors-immo:5-pin-edge-touch, symbol 000-lost-edge-connectors:5-pin-edge-touch
- added J9: i2c-header, 000-edge-connectors-immo:5-pin-edge-touch, symbol 000-lost-edge-connectors:5-pin-edge-touch
- J2: footprint Connector_PCBEdge:BUS_PCIexpress_x1 -> 000-edge-connectors-immo:6-pin-edge-touch; symbol 000-edge-connectors-immo:6-pin-edge-touch -> 000-lost-edge-connectors:6-pin-edge-touch; PIN1 (none) -> SDI; PIN2 (none) -> SDO; PIN3 (none) -> SCK; PIN4 (none) -> SCS; PIN5 (none) -> SWP; PIN6 (none) -> SHD
- J5: symbol 000-edge-connectors-immo:1-pin-edge-touch-XL -> 000-lost-edge-connectors:1-pin-edge-touch-XL; PIN1 (none) -> T0
- J6: symbol 000-edge-connectors-immo:8-pin-edge-touch -> 000-lost-edge-connectors:8-pin-edge-touch; PIN1 (none) -> T2; PIN2 (none) -> T3; PIN3 (none) -> T4; PIN4 (none) -> T5; PIN5 (none) -> T6; PIN6 (none) -> T7; PIN7 (none) -> T8; PIN8 (none) -> T9
Connections:
- net +5V_IN: now also J9.A5
- net 18: now also U3.30 (GPIO18), J4.A3
- net 19: now also J4.A4
- net 23: now also D1.2 (A), U3.37 (GPIO23), J4.A5
- net 3V3_OUT: now also J4.A2, J9.A4
- net GND: now also J4.A1, J9.A1
- net SCL: now also J9.A2
- net SDA: now also J9.A3
- net at U3.4 (SENSOR_VP): now also J10.A1
- net at U3.5 (SENSOR_VN): now also J10.A2
- net at U3.6 (IO34): now also J10.A3
- net at U3.7 (IO35): now also J10.A4
Other:
- moved on the sheet: R8, R9

Commit message: desgfdfg
Parts:
- J10: symbol 000-lost-edge-connectors:4-pin-edge-touch -> 000-edge-connectors-immo:4-pin-edge-touch
- J2: symbol 000-lost-edge-connectors:6-pin-edge-touch -> 000-edge-connectors-immo:6-pin-edge-touch
- J4, J9: symbol 000-lost-edge-connectors:5-pin-edge-touch -> 000-edge-connectors-immo:5-pin-edge-touch
- J5: symbol 000-lost-edge-connectors:1-pin-edge-touch-XL -> 000-edge-connectors-immo:1-pin-edge-touch-XL
- J6: symbol 000-lost-edge-connectors:8-pin-edge-touch -> 000-edge-connectors-immo:8-pin-edge-touch
Changed lines of the file:
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@@
     (effects (font (size 1.27 1.27)) (justify left))
   )
-  (symbol (lib_id "000-lost-edge-connectors:1-pin-edge-touch-XL") (at 200.66 115.57 0) (unit 1)
+  (symbol (lib_id "000-edge-connectors-immo:1-pin-edge-touch-XL") (at 200.66 115.57 0) (unit 1)
     (in_bom yes) (on_board yes) (dnp no)
     (property "Reference" "J5" (at 190.5 94.615 0)
@@
     )
   )
-  (symbol (lib_id "000-lost-edge-connectors:5-pin-edge-touch") (at 257.175 146.685 0) (mirror x) (unit 1)
+  (symbol (lib_id "000-edge-connectors-immo:5-pin-edge-touch") (at 257.175 146.685 0) (mirror x) (unit 1)
     (in_bom yes) (on_board yes) (dnp no)
     (property "Reference" "J9" (at 250.19 146.05 0)
@@
     )
   )
-  (symbol (lib_id "000-lost-edge-connectors:4-pin-edge-touch") (at 100.33 96.52 0) (mirror y) (unit 1)
+  (symbol (lib_id "000-edge-connectors-immo:4-pin-edge-touch") (at 100.33 96.52 0) (mirror y) (unit 1)
     (in_bom yes) (on_board yes) (dnp no)
     (property "Reference" "J10" (at 103.505 74.93 0)
@@
       (effects (font (size 1.27 1.27)))
     )
-    (property "PIN3" "34" (at 93.98 86.995 0)
-      (effects (font (size 1.27 1.27)))
-    )
-    (property "PIN4" "35" (at 93.98 88.9 0)
+    (property "PIN3" "34" (at 93.345 86.36 0)
+      (effects (font (size 1.27 1.27)))
+    )
+    (property "PIN4" "35" (at 93.345 88.265 0)
       (effects (font (size 1.27 1.27)))
     )
@@
     )
   )
-  (symbol (lib_id "000-lost-edge-connectors:8-pin-edge-touch") (at 200.66 127 0) (unit 1)
+  (symbol (lib_id "000-edge-connectors-immo:8-pin-edge-touch") (at 200.66 127 0) (unit 1)
     (in_bom yes) (on_board yes) (dnp no)
     (property "Reference" "J6" (at 194.31 135.89 0)
@@
     )
   )
-  (symbol (lib_id "000-lost-edge-connectors:6-pin-edge-touch") (at 100.33 118.11 0) (mirror y) (unit 1)
+  (symbol (lib_id "000-edge-connectors-immo:6-pin-edge-touch") (at 100.33 118.11 0) (mirror y) (unit 1)
     (in_bom yes) (on_board yes) (dnp no)
     (property "Reference" "J2" (at 103.505 96.52 0)
@@
     )
   )
-  (symbol (lib_id "000-lost-edge-connectors:5-pin-edge-touch") (at 106.68 166.37 180) (unit 1)
+  (symbol (lib_id "000-edge-connectors-immo:5-pin-edge-touch") (at 106.68 166.37 180) (unit 1)
     (in_bom yes) (on_board yes) (dnp no)
     (property "Reference" "J4" (at 113.665 166.37 0)

Commit message: 34terg
Parts:
- added D2, D3: BZV55B3V3, Diode_SMD:D_MiniMELF, symbol Diode:BZV55B3V3
- added J7: DAC/ADC, 000-edge-connectors-immo:4-pin-edge, symbol 000-edge-connectors-immo:4-pin-edge-touch
- added R13, R14: 220r, Resistor_SMD:R_0805_2012Metric_Pad1.20x1.40mm_HandSolder, symbol 000_Resistors_Immo:Resistor_0805
- added R15, R16: 100r, Resistor_SMD:R_0805_2012Metric_Pad1.20x1.40mm_HandSolder, symbol 000_Resistors_Immo:Resistor_0805
Connections:
- net 3V3_OUT: now also J7.A2
- net GND: now also J7.A1, R15.1, R16.1
- net at U3.10 (GPIO25(DAC_1)): now also R13.2
- net at U3.11 (GPIO26(DAC_2)): now also R14.2
- new net: D2.1 (K), J7.A3, R14.1
- new net: D2.2 (A), R16.2
- new net: D3.1 (K), J7.A4, R13.1
- new net: D3.2 (A), R15.2
Other:
- note added: "overvoltage protection. Install when using ADC function, or as protection from external devices"
