File: ISOpower_ESP32.kicad_sch (KiCad schematic)
At the start: 24 parts, among them J10 ESPpin1-4, J2 SDI/SDO, J4 gpio-B, J5 touch0, J6 Touch Pins, J7 DAC/ADC, J9 i2c-header, U2 AMS1117-3.3, U3 ESP32-WROOM-32

Commit message: Adding BOM
Parts:
- C2, C3, C4, C5: footprint Capacitor_SMD:C_0805_2012Metric_Pad1.18x1.45mm_HandSolder -> 000_Capacitors_Immo:C_0805_2012_HandSolder_kawaii; symbol 000_Capacitor_Film_Immo:cap_film_0805 -> 000_Capacitor_Film_Immo:100n; Cost (none) -> 0.02; JLCpart (none) -> C779975
- R8, R9: symbol 000_Resistors_Immo:Resistor_0805 -> 000_Resistors_Immo:10k; Cost (none) -> 0.002; JLCpart (none) -> C2930231
Connections:
- net 3V3_OUT: no longer R8.1, R9.1
- net SCL: no longer R8.2
- net SDA: no longer R9.2
Changed lines of the file:
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@@
     )
   )
-  (symbol (lib_id "000_Resistors_Immo:Resistor_0805") (at 224.155 151.765 0) (unit 1)
+  (symbol (lib_id "000_Resistors_Immo:10k") (at 224.155 151.765 0) (unit 1)
     (in_bom yes) (on_board yes) (dnp no)
     (property "Reference" "R9" (at 219.075 150.495 0)
@@
       (effects (font (size 1.27 1.27)) (justify left))
     )
-    (property "Footprint" "Resistor_SMD:R_0805_2012Metric_Pad1.20x1.40mm_HandSolder" (at 222.377 151.765 90)
-      (effects (font (size 1.27 1.27)) hide)
-    )
-    (property "Datasheet" "~" (at 224.155 151.765 0)
+    (property "Footprint" "Resistor_SMD:R_0805_2012Metric_Pad1.20x1.40mm_HandSolder" (at 224.155 153.543 0)
+      (effects (font (size 1.27 1.27)) hide)
+    )
+    (property "Datasheet" "~" (at 224.155 151.765 90)
+      (effects (font (size 1.27 1.27)) hide)
+    )
+    (property "JLCpart" "C2930231" (at 225.425 154.305 0)
+      (effects (font (size 1.27 1.27)) hide)
+    )
+    (property "Cost" "0.002" (at 224.155 154.305 0)
       (effects (font (size 1.27 1.27)) hide)
     )
@@
     )
   )
-  (symbol (lib_id "000_Capacitor_Film_Immo:cap_film_0805") (at 57.15 35.56 0) (unit 1)
+  (symbol (lib_id "000_Capacitor_Film_Immo:100n") (at 57.15 35.56 0) (unit 1)
     (in_bom yes) (on_board yes) (dnp no) (fields_autoplaced)
-    (property "Reference" "C2" (at 60.96 34.2899 0)
-      (effects (font (size 1.27 1.27)) (justify left))
-    )
-    (property "Value" "100n" (at 60.96 36.8299 0)
-      (effects (font (size 1.27 1.27)) (justify left))
-    )
-    (property "Footprint" "Capacitor_SMD:C_0805_2012Metric_Pad1.18x1.45mm_HandSolder" (at 58.42 45.72 0)
+    (property "Reference" "C2" (at 60.96 34.925 0)
+      (effects (font (size 1.27 1.27)) (justify left))
+    )
+    (property "Value" "100n" (at 60.96 37.465 0)
+      (effects (font (size 1.27 1.27)) (justify left))
+    )
+    (property "Footprint" "000_Capacitors_Immo:C_0805_2012_HandSolder_kawaii" (at 58.42 45.72 0)
       (effects (font (size 1.27 1.27)) hide)
     )
     (property "Datasheet" "~" (at 57.15 35.56 0)
+      (effects (font (size 1.27 1.27)) hide)
+    )
+    (property "JLCpart" "C779975" (at 58.42 45.72 0)
+      (effects (font (size 1.27 1.27)) hide)
+    )
+    (property "Cost" "0.02" (at 60.96 45.72 0)
       (effects (font (size 1.27 1.27)) hide)
     )
@@
     )
   )
-  (symbol (lib_id "000_Capacitor_Film_Immo:cap_film_0805") (at 83.82 35.56 0) (unit 1)
+  (symbol (lib_id "000_Capacitor_Film_Immo:100n") (at 83.82 35.56 0) (unit 1)
     (in_bom yes) (on_board yes) (dnp no) (fields_autoplaced)
-    (property "Reference" "C3" (at 87.63 34.2899 0)
-      (effects (font (size 1.27 1.27)) (justify left))
-    )
-    (property "Value" "100n" (at 87.63 36.8299 0)
-      (effects (font (size 1.27 1.27)) (justify left))
-    )
-    (property "Footprint" "Capacitor_SMD:C_0805_2012Metric_Pad1.18x1.45mm_HandSolder" (at 85.09 45.72 0)
+    (property "Reference" "C3" (at 87.63 34.925 0)
+      (effects (font (size 1.27 1.27)) (justify left))
+    )
+    (property "Value" "100n" (at 87.63 37.465 0)
+      (effects (font (size 1.27 1.27)) (justify left))
+    )
+    (property "Footprint" "000_Capacitors_Immo:C_0805_2012_HandSolder_kawaii" (at 85.09 45.72 0)
       (effects (font (size 1.27 1.27)) hide)
     )
@@
       (effects (font (size 1.27 1.27)) hide)
     )
+    (property "JLCpart" "C779975" (at 85.09 45.72 0)
+      (effects (font (size 1.27 1.27)) hide)
+    )
+    (property "Cost" "0.02" (at 87.63 45.72 0)
+      (effects (font (size 1.27 1.27)) hide)
+    )
     (pin "1")
     (pin "2")
@@
     )
   )
-  (symbol (lib_id "000_Capacitor_Film_Immo:cap_film_0805") (at 116.84 59.69 0) (unit 1)
+  (symbol (lib_id "000_Capacitor_Film_Immo:100n") (at 116.84 59.69 0) (unit 1)
     (in_bom yes) (on_board yes) (dnp no)
     (property "Reference" "C4" (at 118.11 57.15 0)
@@
       (effects (font (size 1.27 1.27)) (justify left))
     )
-    (property "Footprint" "Capacitor_SMD:C_0805_2012Metric_Pad1.18x1.45mm_HandSolder" (at 118.11 69.85 0)
+    (property "Footprint" "000_Capacitors_Immo:C_0805_2012_HandSolder_kawaii" (at 118.11 69.85 0)
       (effects (font (size 1.27 1.27)) hide)
     )
@@
       (effects (font (size 1.27 1.27)) hide)
     )
+    (property "JLCpart" "C779975" (at 118.11 69.85 0)
+      (effects (font (size 1.27 1.27)) hide)
+    )
+    (property "Cost" "0.02" (at 120.65 69.85 0)
+      (effects (font (size 1.27 1.27)) hide)
+    )
     (pin "1")
     (pin "2")
@@
     )
   )
-  (symbol (lib_id "000_Resistors_Immo:Resistor_0805") (at 206.375 151.765 0) (unit 1)
+  (symbol (lib_id "000_Resistors_Immo:10k") (at 206.375 151.765 0) (unit 1)
     (in_bom yes) (on_board yes) (dnp no)
     (property "Reference" "R8" (at 202.565 150.495 0)
@@
       (effects (font (size 1.27 1.27)) (justify left))
     )
-    (property "Footprint" "Resistor_SMD:R_0805_2012Metric_Pad1.20x1.40mm_HandSolder" (at 204.597 151.765 90)
-      (effects (font (size 1.27 1.27)) hide)
-    )
-    (property "Datasheet" "~" (at 206.375 151.765 0)
+    (property "Footprint" "Resistor_SMD:R_0805_2012Metric_Pad1.20x1.40mm_HandSolder" (at 206.375 153.543 0)
+      (effects (font (size 1.27 1.27)) hide)
+    )
+    (property "Datasheet" "~" (at 206.375 151.765 90)
+      (effects (font (size 1.27 1.27)) hide)
+    )
+    (property "JLCpart" "C2930231" (at 207.645 154.305 0)
+      (effects (font (size 1.27 1.27)) hide)
+    )
+    (property "Cost" "0.002" (at 206.375 154.305 0)
       (effects (font (size 1.27 1.27)) hide)
     )
@@
     )
   )
-  (symbol (lib_id "000_Capacitor_Film_Immo:cap_film_0805") (at 125.73 59.69 0) (unit 1)
+  (symbol (lib_id "000_Capacitor_Film_Immo:100n") (at 125.73 59.69 0) (unit 1)
     (in_bom yes) (on_board yes) (dnp no)
     (property "Reference" "C5" (at 127 57.15 0)
@@
       (effects (font (size 1.27 1.27)))
     )
-    (property "Footprint" "Capacitor_SMD:C_0805_2012Metric_Pad1.18x1.45mm_HandSolder" (at 127 69.85 0)
+    (property "Footprint" "000_Capacitors_Immo:C_0805_2012_HandSolder_kawaii" (at 127 69.85 0)
       (effects (font (size 1.27 1.27)) hide)
     )
@@
       (effects (font (size 1.27 1.27)) hide)
     )
+    (property "JLCpart" "C779975" (at 127 69.85 0)
+      (effects (font (size 1.27 1.27)) hide)
+    )
+    (property "Cost" "0.02" (at 129.54 69.85 0)
+      (effects (font (size 1.27 1.27)) hide)
+    )
