File: ch340_ESP32.kicad_sch (KiCad schematic)
At the start: 9 parts, among them Q19 BC817, Q20 BC817, SW2 BOOT, SW3 EN, U14 CH340C

Commit message: kjsaofklihsdof
Parts:
- renumbered C28 to C6, C29 to C7, Q19 to Q1, Q20 to Q2, R25 to R10, R26 to R11, U14 to U4
Changed lines of the file:
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@@
   (symbol (lib_id "000_Capacitor_Film_Immo:cap_film_0805") (at 127 66.04 270) (mirror x) (unit 1)
     (in_bom yes) (on_board yes) (dnp no)
-    (property "Reference" "C28" (at 129.54 64.77 90)
+    (property "Reference" "C6" (at 129.54 64.77 90)
       (effects (font (size 1.27 1.27)))
     )
@@
       (project "ImogenWren"
         (path "/84b7ad53-68b5-40da-9777-f5bb9a09ecb4/9cdb06a8-babb-4d9b-a75e-e6e2cfc518a0/b86764a3-50e0-4d6c-869d-b8d48d944fad"
-          (reference "C28") (unit 1)
+          (reference "C6") (unit 1)
         )
       )
@@
   (symbol (lib_id "Interface_USB:CH340C") (at 135.89 87.63 0) (unit 1)
     (in_bom yes) (on_board yes) (dnp no) (fields_autoplaced)
-    (property "Reference" "U14" (at 135.3694 102.87 0)
+    (property "Reference" "U4" (at 135.3694 102.87 0)
       (effects (font (size 1.27 1.27)) (justify right))
     )
@@
       (project "ImogenWren"
         (path "/84b7ad53-68b5-40da-9777-f5bb9a09ecb4/9cdb06a8-babb-4d9b-a75e-e6e2cfc518a0/b86764a3-50e0-4d6c-869d-b8d48d944fad"
-          (reference "U14") (unit 1)
+          (reference "U4") (unit 1)
         )
       )
@@
   (symbol (lib_id "000_Capacitor_Film_Immo:cap_film_0805") (at 127 71.12 270) (mirror x) (unit 1)
     (in_bom yes) (on_board yes) (dnp no)
-    (property "Reference" "C29" (at 129.54 69.85 90)
+    (property "Reference" "C7" (at 129.54 69.85 90)
       (effects (font (size 1.27 1.27)))
     )
@@
       (project "ImogenWren"
         (path "/84b7ad53-68b5-40da-9777-f5bb9a09ecb4/9cdb06a8-babb-4d9b-a75e-e6e2cfc518a0/b86764a3-50e0-4d6c-869d-b8d48d944fad"
-          (reference "C29") (unit 1)
+          (reference "C7") (unit 1)
         )
       )
@@
   (symbol (lib_id "Transistor_BJT:BC817") (at 182.88 88.9 0) (unit 1)
     (in_bom yes) (on_board yes) (dnp no) (fields_autoplaced)
-    (property "Reference" "Q19" (at 187.96 87.6299 0)
+    (property "Reference" "Q1" (at 187.96 87.6299 0)
       (effects (font (size 1.27 1.27)) (justify left))
     )
@@
       (project "ImogenWren"
         (path "/84b7ad53-68b5-40da-9777-f5bb9a09ecb4/9cdb06a8-babb-4d9b-a75e-e6e2cfc518a0/b86764a3-50e0-4d6c-869d-b8d48d944fad"
-          (reference "Q19") (unit 1)
+          (reference "Q1") (unit 1)
         )
       )
@@
   (symbol (lib_id "000_Resistors_Immo:Resistor_0805") (at 168.91 88.9 90) (unit 1)
     (in_bom yes) (on_board yes) (dnp no)
-    (property "Reference" "R25" (at 168.91 86.36 90)
+    (property "Reference" "R10" (at 168.91 86.36 90)
       (effects (font (size 1.27 1.27)))
     )
@@
       (project "ImogenWren"
         (path "/84b7ad53-68b5-40da-9777-f5bb9a09ecb4/9cdb06a8-babb-4d9b-a75e-e6e2cfc518a0/b86764a3-50e0-4d6c-869d-b8d48d944fad"
-          (reference "R25") (unit 1)
+          (reference "R10") (unit 1)
         )
       )
@@
   (symbol (lib_id "000_Resistors_Immo:Resistor_0805") (at 168.91 104.14 90) (unit 1)
     (in_bom yes) (on_board yes) (dnp no)
-    (property "Reference" "R26" (at 168.91 101.6 90)
+    (property "Reference" "R11" (at 168.91 101.6 90)
       (effects (font (size 1.27 1.27)))
     )
@@
       (project "ImogenWren"
         (path "/84b7ad53-68b5-40da-9777-f5bb9a09ecb4/9cdb06a8-babb-4d9b-a75e-e6e2cfc518a0/b86764a3-50e0-4d6c-869d-b8d48d944fad"
-          (reference "R26") (unit 1)
+          (reference "R11") (unit 1)
         )
       )
@@
   (symbol (lib_id "Transistor_BJT:BC817") (at 182.88 104.14 0) (mirror x) (unit 1)
     (in_bom yes) (on_board yes) (dnp no) (fields_autoplaced)
-    (property "Reference" "Q20" (at 187.96 102.8699 0)
+    (property "Reference" "Q2" (at 187.96 102.8699 0)
       (effects (font (size 1.27 1.27)) (justify left))
     )
@@
       (project "ImogenWren"
         (path "/84b7ad53-68b5-40da-9777-f5bb9a09ecb4/9cdb06a8-babb-4d9b-a75e-e6e2cfc518a0/b86764a3-50e0-4d6c-869d-b8d48d944fad"
-          (reference "Q20") (unit 1)
-        )
-      )
+          (reference "Q2") (unit 1)
+        )
+      )

Commit message: Adding BOM
Parts:
- C6, C7: footprint Capacitor_SMD:C_0805_2012Metric_Pad1.18x1.45mm_HandSolder -> 000_Capacitors_Immo:C_0805_2012_HandSolder_kawaii; symbol 000_Capacitor_Film_Immo:cap_film_0805 -> 000_Capacitor_Film_Immo:100n; Cost (none) -> 0.02; JLCpart (none) -> C779975
- R10, R11: symbol 000_Resistors_Immo:Resistor_0805 -> 000_Resistors_Immo:10k; Cost (none) -> 0.002; JLCpart (none) -> C2930231
Connections:
- net at Q1.2 (E), U4.13 (~{DTR}): no longer R11.1
- net at Q2.2 (E), U4.14 (~{RTS}): no longer R10.1
- net at Q1.1 (B): no longer R10.2
- net at R11.2: no longer Q2.1 (B)
Changed lines of the file:
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@@
     (effects (font (size 1.27 1.27)) (justify left))
   )
-  (symbol (lib_id "000_Capacitor_Film_Immo:cap_film_0805") (at 127 66.04 270) (mirror x) (unit 1)
+  (symbol (lib_id "000_Capacitor_Film_Immo:100n") (at 127 66.04 270) (mirror x) (unit 1)
     (in_bom yes) (on_board yes) (dnp no)
     (property "Reference" "C6" (at 129.54 64.77 90)
@@
       (effects (font (size 1.27 1.27)))
     )
-    (property "Footprint" "Capacitor_SMD:C_0805_2012Metric_Pad1.18x1.45mm_HandSolder" (at 116.84 64.77 0)
+    (property "Footprint" "000_Capacitors_Immo:C_0805_2012_HandSolder_kawaii" (at 116.84 64.77 0)
       (effects (font (size 1.27 1.27)) hide)
     )
     (property "Datasheet" "~" (at 127 66.04 0)
+      (effects (font (size 1.27 1.27)) hide)
+    )
+    (property "JLCpart" "C779975" (at 116.84 64.77 0)
+      (effects (font (size 1.27 1.27)) hide)
+    )
+    (property "Cost" "0.02" (at 116.84 62.23 0)
       (effects (font (size 1.27 1.27)) hide)
     )
@@
     )
   )
-  (symbol (lib_id "000_Capacitor_Film_Immo:cap_film_0805") (at 127 71.12 270) (mirror x) (unit 1)
+  (symbol (lib_id "000_Capacitor_Film_Immo:100n") (at 127 71.12 270) (mirror x) (unit 1)
     (in_bom yes) (on_board yes) (dnp no)
     (property "Reference" "C7" (at 129.54 69.85 90)
@@
       (effects (font (size 1.27 1.27)))
     )
-    (property "Footprint" "Capacitor_SMD:C_0805_2012Metric_Pad1.18x1.45mm_HandSolder" (at 116.84 69.85 0)
+    (property "Footprint" "000_Capacitors_Immo:C_0805_2012_HandSolder_kawaii" (at 116.84 69.85 0)
       (effects (font (size 1.27 1.27)) hide)
     )
     (property "Datasheet" "~" (at 127 71.12 0)
+      (effects (font (size 1.27 1.27)) hide)
+    )
+    (property "JLCpart" "C779975" (at 116.84 69.85 0)
+      (effects (font (size 1.27 1.27)) hide)
+    )
+    (property "Cost" "0.02" (at 116.84 67.31 0)
       (effects (font (size 1.27 1.27)) hide)
     )
@@
     )
   )
-  (symbol (lib_id "000_Resistors_Immo:Resistor_0805") (at 168.91 88.9 90) (unit 1)
+  (symbol (lib_id "000_Resistors_Immo:10k") (at 168.91 88.9 90) (unit 1)
     (in_bom yes) (on_board yes) (dnp no)
     (property "Reference" "R10" (at 168.91 86.36 90)
@@
       (effects (font (size 1.27 1.27)))
     )
-    (property "Footprint" "Resistor_SMD:R_0805_2012Metric_Pad1.20x1.40mm_HandSolder" (at 168.91 90.678 90)
+    (property "Footprint" "Resistor_SMD:R_0805_2012Metric_Pad1.20x1.40mm_HandSolder" (at 170.688 88.9 0)
       (effects (font (size 1.27 1.27)) hide)
     )
-    (property "Datasheet" "~" (at 168.91 88.9 0)
+    (property "Datasheet" "~" (at 168.91 88.9 90)
+      (effects (font (size 1.27 1.27)) hide)
+    )
+    (property "JLCpart" "C2930231" (at 171.45 87.63 0)
+      (effects (font (size 1.27 1.27)) hide)
+    )
+    (property "Cost" "0.002" (at 171.45 88.9 0)
       (effects (font (size 1.27 1.27)) hide)
     )
@@
     )
   )
-  (symbol (lib_id "000_Resistors_Immo:Resistor_0805") (at 168.91 104.14 90) (unit 1)
+  (symbol (lib_id "000_Resistors_Immo:10k") (at 168.91 104.14 90) (unit 1)
     (in_bom yes) (on_board yes) (dnp no)
     (property "Reference" "R11" (at 168.91 101.6 90)
@@
       (effects (font (size 1.27 1.27)))
     )
-    (property "Footprint" "Resistor_SMD:R_0805_2012Metric_Pad1.20x1.40mm_HandSolder" (at 168.91 105.918 90)
+    (property "Footprint" "Resistor_SMD:R_0805_2012Metric_Pad1.20x1.40mm_HandSolder" (at 170.688 104.14 0)
       (effects (font (size 1.27 1.27)) hide)
     )
-    (property "Datasheet" "~" (at 168.91 104.14 0)
+    (property "Datasheet" "~" (at 168.91 104.14 90)
       (effects (font (size 1.27 1.27)) hide)
     )
+    (property "JLCpart" "C2930231" (at 171.45 102.87 0)
+      (effects (font (size 1.27 1.27)) hide)
+    )
+    (property "Cost" "0.002" (at 171.45 104.14 0)
+      (effects (font (size 1.27 1.27)) hide)
+    )
