File: USB-C.kicad_sch (KiCad schematic)
At the start: 8 parts, among them J1 USB_C_Receptacle

Commit message: kjsaofklihsdof
Parts:
- renumbered C1 to C?, C2 to C?, C5 to C?, C4 to C?, C3 to C?, FB1 to FB?, J1 to J?, R1 to R?
Changed lines of the file:
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@@
   (symbol (lib_id "Connector:USB_C_Receptacle") (at 97.79 76.2 0) (unit 1)
     (in_bom yes) (on_board yes) (dnp no) (fields_autoplaced)
-    (property "Reference" "J1" (at 97.79 44.45 0)
+    (property "Reference" "J?" (at 97.79 44.45 0)
       (effects (font (size 1.27 1.27)))
     )
@@
       (project "ImogenWren"
         (path "/84b7ad53-68b5-40da-9777-f5bb9a09ecb4"
-          (reference "J1") (unit 1)
-        )
-        (path "/84b7ad53-68b5-40da-9777-f5bb9a09ecb4/5d70f0ae-944c-460c-8592-0cd073646a17"
-          (reference "J1") (unit 1)
+          (reference "J?") (unit 1)
+        )
+        (path "/84b7ad53-68b5-40da-9777-f5bb9a09ecb4/5d70f0ae-944c-460c-8592-0cd073646a17"
+          (reference "J8") (unit 1)
         )
       )
@@
   (symbol (lib_id "000_Capacitor_Film_Immo:cap_film_0805") (at 130.81 107.95 0) (unit 1)
     (in_bom yes) (on_board yes) (dnp no) (fields_autoplaced)
-    (property "Reference" "C1" (at 134.62 107.315 0)
+    (property "Reference" "C?" (at 134.62 107.315 0)
       (effects (font (size 1.27 1.27)) (justify left))
     )
@@
       (project "ImogenWren"
         (path "/84b7ad53-68b5-40da-9777-f5bb9a09ecb4"
-          (reference "C1") (unit 1)
-        )
-        (path "/84b7ad53-68b5-40da-9777-f5bb9a09ecb4/5d70f0ae-944c-460c-8592-0cd073646a17"
-          (reference "C4") (unit 1)
+          (reference "C?") (unit 1)
+        )
+        (path "/84b7ad53-68b5-40da-9777-f5bb9a09ecb4/5d70f0ae-944c-460c-8592-0cd073646a17"
+          (reference "C8") (unit 1)
         )
       )
@@
   (symbol (lib_id "000_Resistors_Immo:Resistor_0805") (at 120.65 107.95 90) (unit 1)
     (in_bom yes) (on_board yes) (dnp no) (fields_autoplaced)
-    (property "Reference" "R1" (at 123.19 107.315 90)
+    (property "Reference" "R?" (at 123.19 107.315 90)
       (effects (font (size 1.27 1.27)) (justify right))
     )
@@
       (project "ImogenWren"
         (path "/84b7ad53-68b5-40da-9777-f5bb9a09ecb4"
-          (reference "R1") (unit 1)
-        )
-        (path "/84b7ad53-68b5-40da-9777-f5bb9a09ecb4/5d70f0ae-944c-460c-8592-0cd073646a17"
-          (reference "R1") (unit 1)
+          (reference "R?") (unit 1)
+        )
+        (path "/84b7ad53-68b5-40da-9777-f5bb9a09ecb4/5d70f0ae-944c-460c-8592-0cd073646a17"
+          (reference "R12") (unit 1)
         )
       )
@@
   (symbol (lib_id "power:GNDPWR") (at 149.86 53.34 0) (unit 1)
     (in_bom yes) (on_board yes) (dnp no) (fields_autoplaced)
-    (property "Reference" "#PWR02" (at 149.86 58.42 0)
+    (property "Reference" "#PWR?" (at 149.86 58.42 0)
       (effects (font (size 1.27 1.27)) hide)
     )
@@
       (project "ImogenWren"
         (path "/84b7ad53-68b5-40da-9777-f5bb9a09ecb4"
-          (reference "#PWR02") (unit 1)
-        )
-        (path "/84b7ad53-68b5-40da-9777-f5bb9a09ecb4/5d70f0ae-944c-460c-8592-0cd073646a17"
-          (reference "#PWR02") (unit 1)
+          (reference "#PWR?") (unit 1)
+        )
+        (path "/84b7ad53-68b5-40da-9777-f5bb9a09ecb4/5d70f0ae-944c-460c-8592-0cd073646a17"
+          (reference "#PWR06") (unit 1)
         )
       )
@@
   (symbol (lib_id "Device:FerriteBead") (at 138.43 50.8 90) (unit 1)
     (in_bom yes) (on_board yes) (dnp no) (fields_autoplaced)
-    (property "Reference" "FB1" (at 138.3792 44.45 90)
+    (property "Reference" "FB?" (at 138.3792 44.45 90)
       (effects (font (size 1.27 1.27)))
     )
@@
       (project "ImogenWren"
         (path "/84b7ad53-68b5-40da-9777-f5bb9a09ecb4"
+          (reference "FB?") (unit 1)
+        )
+        (path "/84b7ad53-68b5-40da-9777-f5bb9a09ecb4/5d70f0ae-944c-460c-8592-0cd073646a17"
           (reference "FB1") (unit 1)
         )
-        (path "/84b7ad53-68b5-40da-9777-f5bb9a09ecb4/5d70f0ae-944c-460c-8592-0cd073646a17"
-          (reference "FB1") (unit 1)
-        )
       )
     )
@@
   (symbol (lib_id "power:GNDPWR") (at 161.29 53.34 0) (unit 1)
     (in_bom yes) (on_board yes) (dnp no) (fields_autoplaced)
-    (property "Reference" "#PWR03" (at 161.29 58.42 0)
+    (property "Reference" "#PWR?" (at 161.29 58.42 0)
       (effects (font (size 1.27 1.27)) hide)
     )
@@
       (project "ImogenWren"
         (path "/84b7ad53-68b5-40da-9777-f5bb9a09ecb4"
-          (reference "#PWR03") (unit 1)
-        )
-        (path "/84b7ad53-68b5-40da-9777-f5bb9a09ecb4/5d70f0ae-944c-460c-8592-0cd073646a17"
-          (reference "#PWR03") (unit 1)
+          (reference "#PWR?") (unit 1)
+        )
+        (path "/84b7ad53-68b5-40da-9777-f5bb9a09ecb4/5d70f0ae-944c-460c-8592-0cd073646a17"
+          (reference "#PWR07") (unit 1)
         )
       )
@@
   (symbol (lib_id "000_Capacitor_Film_Immo:cap_film_0805") (at 149.86 46.99 0) (unit 1)
     (in_bom yes) (on_board yes) (dnp no) (fields_autoplaced)
-    (property "Reference" "C2" (at 153.67 46.355 0)
+    (property "Reference" "C?" (at 153.67 46.355 0)
       (effects (font (size 1.27 1.27)) (justify left))
     )
@@
       (project "ImogenWren"
         (path "/84b7ad53-68b5-40da-9777-f5bb9a09ecb4"
-          (reference "C2") (unit 1)
-        )
-        (path "/84b7ad53-68b5-40da-9777-f5bb9a09ecb4/5d70f0ae-944c-460c-8592-0cd073646a17"
-          (reference "C13") (unit 1)
+          (reference "C?") (unit 1)
+        )
+        (path "/84b7ad53-68b5-40da-9777-f5bb9a09ecb4/5d70f0ae-944c-460c-8592-0cd073646a17"
+          (reference "C10") (unit 1)
         )
       )
@@
   (symbol (lib_id "000_Capacitor_Film_Immo:cap_film_0805") (at 157.48 107.95 0) (unit 1)
     (in_bom yes) (on_board yes) (dnp no) (fields_autoplaced)
-    (property "Reference" "C5" (at 161.29 107.315 0)
+    (property "Reference" "C?" (at 161.29 107.315 0)
       (effects (font (size 1.27 1.27)) (justify left))
     )
@@
       (project "ImogenWren"
         (path "/84b7ad53-68b5-40da-9777-f5bb9a09ecb4"
-          (reference "C5") (unit 1)
-        )
-        (path "/84b7ad53-68b5-40da-9777-f5bb9a09ecb4/5d70f0ae-944c-460c-8592-0cd073646a17"
-          (reference "C14") (unit 1)
+          (reference "C?") (unit 1)
+        )
+        (path "/84b7ad53-68b5-40da-9777-f5bb9a09ecb4/5d70f0ae-944c-460c-8592-0cd073646a17"
+          (reference "C11") (unit 1)
         )
       )
@@
   (symbol (lib_id "000_Capacitor_Film_Immo:cap_film_0805") (at 146.05 107.95 0) (unit 1)
     (in_bom yes) (on_board yes) (dnp no) (fields_autoplaced)
-    (property "Reference" "C4" (at 149.86 107.315 0)
+    (property "Reference" "C?" (at 149.86 107.315 0)
       (effects (font (size 1.27 1.27)) (justify left))
     )
@@
       (project "ImogenWren"
         (path "/84b7ad53-68b5-40da-9777-f5bb9a09ecb4"
-          (reference "C4") (unit 1)
+          (reference "C?") (unit 1)
+        )
+        (path "/84b7ad53-68b5-40da-9777-f5bb9a09ecb4/5d70f0ae-944c-460c-8592-0cd073646a17"
+          (reference "C9") (unit 1)
+        )
+      )
+    )
+  )
+  (symbol (lib_id "000_Capacitor_Film_Immo:cap_film_0805") (at 161.29 46.99 0) (unit 1)
+    (in_bom yes) (on_board yes) (dnp no) (fields_autoplaced)
+    (property "Reference" "C?" (at 165.1 46.355 0)
+      (effects (font (size 1.27 1.27)) (justify left))
+    )
+    (property "Value" "4n7" (at 165.1 48.895 0)
+      (effects (font (size 1.27 1.27)) (justify left))
+    )
+    (property "Footprint" "Capacitor_SMD:C_0805_2012Metric_Pad1.18x1.45mm_HandSolder" (at 162.56 57.15 0)
+      (effects (font (size 1.27 1.27)) hide)
+    )
+    (property "Datasheet" "~" (at 161.29 46.99 0)
+      (effects (font (size 1.27 1.27)) hide)
+    )
+    (pin "1")
+    (pin "2")
+    (instances
+      (project "ImogenWren"
+        (path "/84b7ad53-68b5-40da-9777-f5bb9a09ecb4"
+          (reference "C?") (unit 1)
         )
         (path "/84b7ad53-68b5-40da-9777-f5bb9a09ecb4/5d70f0ae-944c-460c-8592-0cd073646a17"
@@
         )
       )
-    )
-  )
-  (symbol (lib_id "000_Capacitor_Film_Immo:cap_film_0805") (at 161.29 46.99 0) (unit 1)
-    (in_bom yes) (on_board yes) (dnp no) (fields_autoplaced)
-    (property "Reference" "C3" (at 165.1 46.355 0)
-      (effects (font (size 1.27 1.27)) (justify left))
-    )
-    (property "Value" "4n7" (at 165.1 48.895 0)
-      (effects (font (size 1.27 1.27)) (justify left))
-    )
-    (property "Footprint" "Capacitor_SMD:C_0805_2012Metric_Pad1.18x1.45mm_HandSolder" (at 162.56 57.15 0)
-      (effects (font (size 1.27 1.27)) hide)
-    )
-    (property "Datasheet" "~" (at 161.29 46.99 0)
-      (effects (font (size 1.27 1.27)) hide)
-    )
-    (pin "1")
-    (pin "2")
-    (instances
-      (project "ImogenWren"
-        (path "/84b7ad53-68b5-40da-9777-f5bb9a09ecb4"
-          (reference "C3") (unit 1)
-        )
-        (path "/84b7ad53-68b5-40da-9777-f5bb9a09ecb4/5d70f0ae-944c-460c-8592-0cd073646a17"
-          (reference "C15") (unit 1)
-        )
-      )

Commit message: Adding BOM
Parts:
- C?: footprint Capacitor_SMD:C_0805_2012Metric_Pad1.18x1.45mm_HandSolder -> 000_Capacitors_Immo:C_0805_2012_HandSolder_kawaii; symbol 000_Capacitor_Film_Immo:cap_film_0805 -> 000_Capacitor_Film_Immo:100n; Cost (none) -> 0.02; JLCpart (none) -> C779975
Changed lines of the file:
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@@
     )
   )
-  (symbol (lib_id "000_Capacitor_Film_Immo:cap_film_0805") (at 149.86 46.99 0) (unit 1)
+  (symbol (lib_id "000_Capacitor_Film_Immo:100n") (at 149.86 46.99 0) (unit 1)
     (in_bom yes) (on_board yes) (dnp no) (fields_autoplaced)
     (property "Reference" "C?" (at 153.67 46.355 0)
@@
       (effects (font (size 1.27 1.27)) (justify left))
     )
-    (property "Footprint" "Capacitor_SMD:C_0805_2012Metric_Pad1.18x1.45mm_HandSolder" (at 151.13 57.15 0)
+    (property "Footprint" "000_Capacitors_Immo:C_0805_2012_HandSolder_kawaii" (at 151.13 57.15 0)
       (effects (font (size 1.27 1.27)) hide)
     )
@@
       (effects (font (size 1.27 1.27)) hide)
     )
+    (property "JLCpart" "C779975" (at 151.13 57.15 0)
+      (effects (font (size 1.27 1.27)) hide)
+    )
+    (property "Cost" "0.02" (at 153.67 57.15 0)
+      (effects (font (size 1.27 1.27)) hide)
+    )

Commit message: dfghdfh
Parts:
- FB?: symbol Device:FerriteBead -> 000_inductors_immo:FerriteBead; Cost (none) -> 0.558; JLCpart (none) -> C845115
- J?: symbol Connector:USB_C_Receptacle -> 000_Connectors_Immo:USB_C_Receptacle; Cost (none) -> 0.6619; JLCpart (none) -> C134092
Changed lines of the file:
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@@
     (effects (font (size 1.27 1.27)) (justify left))
   )
-  (symbol (lib_id "Connector:USB_C_Receptacle") (at 97.79 76.2 0) (unit 1)
+  (symbol (lib_id "000_Connectors_Immo:USB_C_Receptacle") (at 97.79 76.2 0) (unit 1)
     (in_bom yes) (on_board yes) (dnp no) (fields_autoplaced)
     (property "Reference" "J?" (at 97.79 44.45 0)
@@
     )
     (property "Datasheet" "https://www.usb.org/sites/default/files/documents/usb_type-c.zip" (at 101.6 76.2 0)
+      (effects (font (size 1.27 1.27)) hide)
+    )
+    (property "JLCpart" "C134092" (at 97.79 76.2 0)
+      (effects (font (size 1.27 1.27)) hide)
+    )
+    (property "Cost" "0.6619" (at 97.79 76.2 0)
       (effects (font (size 1.27 1.27)) hide)
     )
@@
     )
   )
-  (symbol (lib_id "Device:FerriteBead") (at 138.43 50.8 90) (unit 1)
+  (symbol (lib_id "000_inductors_immo:FerriteBead") (at 138.43 50.8 90) (unit 1)
     (in_bom yes) (on_board yes) (dnp no) (fields_autoplaced)
     (property "Reference" "FB?" (at 138.3792 44.45 90)
@@
       (effects (font (size 1.27 1.27)) hide)
     )
+    (property "JLCpart" "C845115" (at 138.43 50.8 0)
+      (effects (font (size 1.27 1.27)) hide)
+    )
+    (property "Cost" "0.558" (at 138.43 50.8 0)
+      (effects (font (size 1.27 1.27)) hide)
+    )

Commit message: dsfgdsfgd
Parts:
- C?: footprint Capacitor_SMD:C_0805_2012Metric_Pad1.18x1.45mm_HandSolder -> 000_Capacitors_Immo:C_0805_2012_HandSolder_kawaii; symbol 000_Capacitor_Film_Immo:cap_film_0805 -> 000_Capacitor_Film_Immo:10n_MLCC; Cost (none) -> 0.0051; JLCpart (none) -> C83170
- C? (x2): footprint Capacitor_SMD:C_0805_2012Metric_Pad1.18x1.45mm_HandSolder -> 000_Capacitors_Immo:C_0805_2012_HandSolder_kawaii; symbol 000_Capacitor_Film_Immo:cap_film_0805 -> 000_Capacitor_Film_Immo:47p_MLCC; Cost (none) -> 0.0056; JLCpart (none) -> C24659
- C?: footprint Capacitor_SMD:C_0805_2012Metric_Pad1.18x1.45mm_HandSolder -> 000_Capacitors_Immo:C_0805_2012_HandSolder_kawaii; symbol 000_Capacitor_Film_Immo:cap_film_0805 -> 000_Capacitor_Film_Immo:4n7_MLCC; Cost (none) -> 0.0118; JLCpart (none) -> C2915753
- R?: value 5k2 -> 4k7; symbol 000_Resistors_Immo:Resistor_0805 -> 000_Resistors_Immo:4k7; Cost (none) -> 0.002; JLCpart (none) -> C5140142
Other:
- note added: "5k2 - unavailable"
Changed lines of the file:
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@@
+    (effects (font (size 1.27 1.27)) (justify left bottom))
+  )
+  (text "5k2 -\nunavailable" (at 121.285 102.87 0)
     (effects (font (size 1.27 1.27)) (justify left bottom))
   )
@@
     )
   )
-  (symbol (lib_id "000_Capacitor_Film_Immo:cap_film_0805") (at 130.81 107.95 0) (unit 1)
+  (symbol (lib_id "000_Capacitor_Film_Immo:10n_MLCC") (at 130.81 107.95 0) (unit 1)
     (in_bom yes) (on_board yes) (dnp no) (fields_autoplaced)
     (property "Reference" "C?" (at 134.62 107.315 0)
@@
       (effects (font (size 1.27 1.27)) (justify left))
     )
-    (property "Footprint" "Capacitor_SMD:C_0805_2012Metric_Pad1.18x1.45mm_HandSolder" (at 132.08 118.11 0)
+    (property "Footprint" "000_Capacitors_Immo:C_0805_2012_HandSolder_kawaii" (at 132.08 118.11 0)
       (effects (font (size 1.27 1.27)) hide)
     )
@@
       (effects (font (size 1.27 1.27)) hide)
     )
+    (property "JLCpart" "C83170" (at 132.08 118.11 0)
+      (effects (font (size 1.27 1.27)) hide)
+    )
+    (property "Cost" "0.0051" (at 134.62 118.11 0)
+      (effects (font (size 1.27 1.27)) hide)
+    )
     (pin "1")
     (pin "2")
@@
     )
   )
-  (symbol (lib_id "000_Resistors_Immo:Resistor_0805") (at 120.65 107.95 90) (unit 1)
+  (symbol (lib_id "000_Resistors_Immo:4k7") (at 120.65 107.95 90) (unit 1)
     (in_bom yes) (on_board yes) (dnp no) (fields_autoplaced)
     (property "Reference" "R?" (at 123.19 107.315 90)
       (effects (font (size 1.27 1.27)) (justify right))
     )
-    (property "Value" "5k2" (at 123.19 109.855 90)
+    (property "Value" "4k7" (at 123.19 109.855 90)
       (effects (font (size 1.27 1.27)) (justify right))
     )
@@
       (effects (font (size 1.27 1.27)) hide)
     )
+    (property "JLCpart" "C5140142" (at 123.19 106.68 0)
+      (effects (font (size 1.27 1.27)) hide)
+    )
+    (property "Cost" "0.002" (at 123.19 107.95 0)
+      (effects (font (size 1.27 1.27)) hide)
+    )
     (pin "1")
     (pin "2")
@@
     )
   )
-  (symbol (lib_id "000_Capacitor_Film_Immo:cap_film_0805") (at 157.48 107.95 0) (unit 1)
+  (symbol (lib_id "000_Capacitor_Film_Immo:47p_MLCC") (at 157.48 107.95 0) (unit 1)
     (in_bom yes) (on_board yes) (dnp no) (fields_autoplaced)
     (property "Reference" "C?" (at 161.29 107.315 0)
@@
       (effects (font (size 1.27 1.27)) (justify left))
     )
-    (property "Footprint" "Capacitor_SMD:C_0805_2012Metric_Pad1.18x1.45mm_HandSolder" (at 158.75 118.11 0)
+    (property "Footprint" "000_Capacitors_Immo:C_0805_2012_HandSolder_kawaii" (at 158.75 118.11 0)
       (effects (font (size 1.27 1.27)) hide)
     )
@@
       (effects (font (size 1.27 1.27)) hide)
     )
+    (property "JLCpart" "C24659" (at 158.75 118.11 0)
+      (effects (font (size 1.27 1.27)) hide)
+    )
+    (property "Cost" "0.0056" (at 161.29 118.11 0)
+      (effects (font (size 1.27 1.27)) hide)
+    )
     (pin "1")
     (pin "2")
@@
     )
   )
-  (symbol (lib_id "000_Capacitor_Film_Immo:cap_film_0805") (at 146.05 107.95 0) (unit 1)
+  (symbol (lib_id "000_Capacitor_Film_Immo:47p_MLCC") (at 146.05 107.95 0) (unit 1)
     (in_bom yes) (on_board yes) (dnp no) (fields_autoplaced)
     (property "Reference" "C?" (at 149.86 107.315 0)
@@
       (effects (font (size 1.27 1.27)) (justify left))
     )
-    (property "Footprint" "Capacitor_SMD:C_0805_2012Metric_Pad1.18x1.45mm_HandSolder" (at 147.32 118.11 0)
+    (property "Footprint" "000_Capacitors_Immo:C_0805_2012_HandSolder_kawaii" (at 147.32 118.11 0)
       (effects (font (size 1.27 1.27)) hide)
     )
@@
       (effects (font (size 1.27 1.27)) hide)
     )
+    (property "JLCpart" "C24659" (at 147.32 118.11 0)
+      (effects (font (size 1.27 1.27)) hide)
+    )
+    (property "Cost" "0.0056" (at 149.86 118.11 0)
+      (effects (font (size 1.27 1.27)) hide)
+    )
     (pin "1")
     (pin "2")
@@
     )
   )
-  (symbol (lib_id "000_Capacitor_Film_Immo:cap_film_0805") (at 161.29 46.99 0) (unit 1)
+  (symbol (lib_id "000_Capacitor_Film_Immo:4n7_MLCC") (at 161.29 46.99 0) (unit 1)
     (in_bom yes) (on_board yes) (dnp no) (fields_autoplaced)
     (property "Reference" "C?" (at 165.1 46.355 0)
@@
       (effects (font (size 1.27 1.27)) (justify left))
     )
-    (property "Footprint" "Capacitor_SMD:C_0805_2012Metric_Pad1.18x1.45mm_HandSolder" (at 162.56 57.15 0)
+    (property "Footprint" "000_Capacitors_Immo:C_0805_2012_HandSolder_kawaii" (at 162.56 57.15 0)
       (effects (font (size 1.27 1.27)) hide)
     )
@@
       (effects (font (size 1.27 1.27)) hide)
     )
+    (property "JLCpart" "C2915753" (at 162.56 57.15 0)
+      (effects (font (size 1.27 1.27)) hide)
+    )
+    (property "Cost" "0.0118" (at 165.1 57.15 0)
+      (effects (font (size 1.27 1.27)) hide)
+    )
