File: pcb-esp32-faerfly/ImogenWren.kicad_sch (KiCad schematic)
At the start: 18 parts, among them J1 LiPo_4v2, J3 WS2821b, SW1 SW_SPDT_small, U1 MCP73831-2-OT

Commit message: Added Complete BOM
Ready for Parts Shopping!
Parts:
- J1, J3, JP1, JP2, JP3, JPw1: now left out of the parts list
- R4, R5: symbol 000_Resistors_Immo:Resistor_0805 -> 000_Resistors_Immo:27r; Cost (none) -> 0.002; JLCpart (none) -> C779975
- U1: symbol Battery_Management:MCP73831-2-OT -> 000_IC_immo:MCP73831-2-OT-batt-management; Cost (none) -> 0.778; JLCpart (none) -> C424093
Changed lines of the file:
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@@
     (effects (font (size 1.27 1.27)) (justify right))
   )
-  (symbol (lib_id "000_Resistors_Immo:Resistor_0805") (at 74.93 83.185 180) (unit 1)
+  (symbol (lib_id "000_Resistors_Immo:27r") (at 74.93 83.185 180) (unit 1)
     (in_bom yes) (on_board yes) (dnp no)
     (property "Reference" "R4" (at 74.93 78.105 0)
@@
       (effects (font (size 1.27 1.27)) hide)
     )
+    (property "JLCpart" "C779975" (at 73.66 80.645 0)
+      (effects (font (size 1.27 1.27)) hide)
+    )
+    (property "Cost" "0.002" (at 74.93 80.645 0)
+      (effects (font (size 1.27 1.27)) hide)
+    )
     (pin "1")
     (pin "2")
@@
   )
   (symbol (lib_id "000_Connectors_Immo:Jumper_3_Bridged12") (at 109.22 39.37 90) (mirror x) (unit 1)
-    (in_bom yes) (on_board yes) (dnp no)
+    (in_bom no) (on_board yes) (dnp no)
     (property "Reference" "JP2" (at 107.95 40.005 90)
       (effects (font (size 1.27 1.27)) (justify left))
@@
   )
   (symbol (lib_id "000_Connectors_Immo:Jumper_2_Bridge_Small") (at 201.295 31.75 0) (unit 1)
-    (in_bom yes) (on_board yes) (dnp no) (fields_autoplaced)
+    (in_bom no) (on_board yes) (dnp no) (fields_autoplaced)
     (property "Reference" "JPw1" (at 201.2725 26.67 0)
       (effects (font (size 1.27 1.27)))
@@
   )
   (symbol (lib_id "Jumper:SolderJumper_3_Open") (at 81.28 171.45 90) (mirror x) (unit 1)
-    (in_bom yes) (on_board yes) (dnp no)
+    (in_bom no) (on_board yes) (dnp no)
     (property "Reference" "JP1" (at 86.36 173.99 90)
       (effects (font (size 1.27 1.27)) (justify left))
@@
   )
   (symbol (lib_id "000_Connectors_Immo:Jumper_3_Bridged12") (at 229.87 73.66 0) (unit 1)
-    (in_bom yes) (on_board yes) (dnp no) (fields_autoplaced)
+    (in_bom no) (on_board yes) (dnp no) (fields_autoplaced)
     (property "Reference" "JP3" (at 229.87 69.85 0)
       (effects (font (size 1.27 1.27)))
@@
   )
   (symbol (lib_id "000-edge-connectors-immo:3-pin-edge-touch") (at 260.35 80.01 0) (mirror x) (unit 1)
-    (in_bom yes) (on_board yes) (dnp no)
+    (in_bom no) (on_board yes) (dnp no)
     (property "Reference" "J3" (at 250.19 87.63 0)
       (effects (font (size 1.27 1.27)) (justify left))
@@
     )
   )
-  (symbol (lib_id "000_Resistors_Immo:Resistor_0805") (at 83.185 88.265 180) (unit 1)
+  (symbol (lib_id "000_Resistors_Immo:27r") (at 83.185 88.265 180) (unit 1)
     (in_bom yes) (on_board yes) (dnp no)
     (property "Reference" "R5" (at 83.185 86.36 0)
@@
       (effects (font (size 1.27 1.27)) hide)
     )
+    (property "JLCpart" "C779975" (at 81.915 85.725 0)
+      (effects (font (size 1.27 1.27)) hide)
+    )
+    (property "Cost" "0.002" (at 83.185 85.725 0)
+      (effects (font (size 1.27 1.27)) hide)
+    )
     (pin "1")
     (pin "2")
@@
     )
   )
-  (symbol (lib_id "Battery_Management:MCP73831-2-OT") (at 87.63 143.51 0) (unit 1)
+  (symbol (lib_id "000_IC_immo:MCP73831-2-OT-batt-management") (at 87.63 143.51 0) (unit 1)
     (in_bom yes) (on_board yes) (dnp no) (fields_autoplaced)
     (property "Reference" "U1" (at 89.5859 134.62 0)
@@
     )
     (property "Datasheet" "http://ww1.microchip.com/downloads/en/DeviceDoc/20001984g.pdf" (at 83.82 144.78 0)
+      (effects (font (size 1.27 1.27)) hide)
+    )
+    (property "JLCpart" "C424093" (at 87.63 143.51 0)
+      (effects (font (size 1.27 1.27)) hide)
+    )
+    (property "Cost" "0.778" (at 87.63 143.51 0)
       (effects (font (size 1.27 1.27)) hide)
     )
@@
   )
   (symbol (lib_id "000-edge-connectors-immo:2-pin-edge-touch") (at 153.035 150.495 0) (mirror x) (unit 1)
-    (in_bom yes) (on_board yes) (dnp no)
+    (in_bom no) (on_board yes) (dnp no)
     (property "Reference" "J1" (at 143.51 143.51 0)
       (effects (font (size 1.27 1.27)) (justify left))
