File: esp32-faerfly-V2.0/ISOpower_ESP32.kicad_sch (KiCad schematic)
At the start: 24 parts, among them J10 ESPpin1-4, J2 SDI/SDO, J4 gpio-B, J5 touch0, J6 Touch Pins, J7 DAC/ADC, J9 i2c-header, U2 AMS1117-3.3, U3 ESP32-WROOM-32

Commit message: Updates to V2.0 PCB
Parts:
- added R2: 100k, Resistor_SMD:R_0805_2012Metric_Pad1.20x1.40mm_HandSolder, symbol 000_Resistors_Immo:100k
Connections:
- net at J6.A8, U3.8 (GPIO32(T9)): now also R2.1
- new net BATT_SNIFF: R2.2
Other:
- note removed: "ESP32 has built in bootloader, therefore does not require AVR SPI interface for programming."
Changed lines of the file:
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@@
 (kicad_sch (version 20230121) (generator eeschema)
   (paper "A4")
+  (junction (at 163.195 129.54) (diameter 0) (color 0 0 0 0)
+  )
   (junction (at 224.155 156.845) (diameter 0) (color 0 0 0 0)
   )
@@
     (stroke (width 0) (type default))
   )
+  (wire (pts (xy 175.895 136.525) (xy 173.355 136.525))
+    (stroke (width 0) (type default))
+  )
   (wire (pts (xy 88.9 137.16) (xy 76.2 137.16))
     (stroke (width 0) (type default))
@@
     (stroke (width 0) (type default))
   )
+  (wire (pts (xy 163.195 136.525) (xy 163.195 129.54))
+    (stroke (width 0) (type default))
+  )
   (wire (pts (xy 170.18 63.5) (xy 173.99 63.5))
     (stroke (width 0) (type default))
@@
     (stroke (width 0) (type default))
   )
+  (wire (pts (xy 163.195 129.54) (xy 185.42 129.54))
+    (stroke (width 0) (type default))
+  )
   (wire (pts (xy 135.89 144.78) (xy 135.89 142.24))
     (stroke (width 0) (type default))
@@
     (stroke (width 0) (type default))
   )
-  (wire (pts (xy 156.21 129.54) (xy 185.42 129.54))
+  (wire (pts (xy 156.21 129.54) (xy 163.195 129.54))
     (stroke (width 0) (type default))
   )
@@
   )
   (wire (pts (xy 125.73 55.88) (xy 125.73 53.34))
+    (stroke (width 0) (type default))
+  )
+  (wire (pts (xy 163.195 136.525) (xy 165.735 136.525))
     (stroke (width 0) (type default))
   )
@@
     (effects (font (size 1.27 1.27)) (justify left bottom))
   )
-  (text "ESP32 has built in bootloader,\ntherefore does not require\nAVR SPI interface for\nprogramming."
-    (at 160.02 147.32 0)
-    (effects (font (size 1.27 1.27)) (justify left bottom))
-  )
   (text "#TODO: check voltage on these pins a\nand also function!"
     (at 86.36 95.25 0)
@@
     (effects (font (size 1.27 1.27)) (justify left bottom))
   )
-  (label "BATTERY_BUS" (at 167.64 43.18 0) (fields_autoplaced)
+  (label "POWER_BUS" (at 167.64 43.18 0) (fields_autoplaced)
     (effects (font (size 1.27 1.27)) (justify left bottom))
   )
@@
     (effects (font (size 1.27 1.27)) (justify right bottom))
   )
-  (label "BATTERY_BUS" (at 40.64 27.94 180) (fields_autoplaced)
+  (label "POWER_BUS" (at 40.64 27.94 180) (fields_autoplaced)
     (effects (font (size 1.27 1.27)) (justify right bottom))
   )
@@
     (effects (font (size 1.27 1.27)) (justify left bottom))
   )
-  (label "BATTERY_BUS" (at 229.235 151.765 0) (fields_autoplaced)
-    (effects (font (size 1.27 1.27)) (justify left bottom))
-  )
-  (global_label "SDA" (shape bidirectional) (at 158.75 86.36 0) (fields_autoplaced)
-    (effects (font (size 1.27 1.27)) (justify left))
-    (property "Intersheetrefs" "${INTERSHEET_REFS}" (at 164.7312 86.2806 0)
-      (effects (font (size 1.27 1.27)) (justify left) hide)
-    )
-  )
-  (global_label "SCL" (shape input) (at 200.025 159.385 180) (fields_autoplaced)
-    (effects (font (size 1.27 1.27)) (justify right))
-    (property "Intersheetrefs" "${INTERSHEET_REFS}" (at 194.1043 159.4644 0)
-      (effects (font (size 1.27 1.27)) (justify right) hide)
-    )
+  (label "POWER_BUS" (at 229.235 151.765 0) (fields_autoplaced)
+    (effects (font (size 1.27 1.27)) (justify left bottom))
   )
   (global_label "19" (shape bidirectional) (at 158.75 90.17 0) (fields_autoplaced)
@@
     )
   )
-  (global_label "SCL" (shape output) (at 158.75 78.74 0) (fields_autoplaced)
-    (effects (font (size 1.27 1.27)) (justify left))
-    (property "Intersheetrefs" "${INTERSHEET_REFS}" (at 164.6707 78.6606 0)
-      (effects (font (size 1.27 1.27)) (justify left) hide)
-    )
-  )
-  (global_label "SDA" (shape bidirectional) (at 220.345 156.845 180) (fields_autoplaced)
-    (effects (font (size 1.27 1.27)) (justify right))
-    (property "Intersheetrefs" "${INTERSHEET_REFS}" (at 214.3638 156.7656 0)
-      (effects (font (size 1.27 1.27)) (justify right) hide)
-    )
-  )
   (global_label "18" (shape bidirectional) (at 158.75 92.71 0) (fields_autoplaced)
     (effects (font (size 1.27 1.27)) (justify left))
@@
     )
   )
+  (hierarchical_label "BATT_SNIFF" (shape input) (at 36.195 57.15 180) (fields_autoplaced)
+    (effects (font (size 1.27 1.27)) (justify right))
+  )
   (hierarchical_label "3V3_OUT" (shape output) (at 27.94 35.56 180) (fields_autoplaced)
     (effects (font (size 1.27 1.27)) (justify right))
   )
+  (hierarchical_label "SDA" (shape bidirectional) (at 158.75 86.36 0) (fields_autoplaced)
+    (effects (font (size 1.27 1.27)) (justify left))
+  )
   (hierarchical_label "SSERIAL_TX" (shape input) (at 158.75 100.33 0) (fields_autoplaced)
     (effects (font (size 1.27 1.27)) (justify left))
+  )
+  (hierarchical_label "SDA" (shape bidirectional) (at 220.345 156.845 180) (fields_autoplaced)
+    (effects (font (size 1.27 1.27)) (justify right))
   )
   (hierarchical_label "D+" (shape input) (at 180.34 46.99 180) (fields_autoplaced)
     (effects (font (size 1.27 1.27)) (justify right))
   )
+  (hierarchical_label "SCL" (shape input) (at 200.025 159.385 180) (fields_autoplaced)
+    (effects (font (size 1.27 1.27)) (justify right))
+  )
   (hierarchical_label "D-" (shape output) (at 180.34 49.53 180) (fields_autoplaced)
     (effects (font (size 1.27 1.27)) (justify right))
@@
     (effects (font (size 1.27 1.27)) (justify right))
   )
+  (hierarchical_label "BATT_SNIFF" (shape input) (at 175.895 136.525 0) (fields_autoplaced)
+    (effects (font (size 1.27 1.27)) (justify left))
+  )
   (hierarchical_label "SSERIAL_RX" (shape output) (at 93.98 76.835 0) (fields_autoplaced)
     (effects (font (size 1.27 1.27)) (justify left))
@@
   )
   (hierarchical_label "SSERIAL_TX" (shape input) (at 93.98 79.375 0) (fields_autoplaced)
+    (effects (font (size 1.27 1.27)) (justify left))
+  )
+  (hierarchical_label "SCL" (shape output) (at 158.75 78.74 0) (fields_autoplaced)
     (effects (font (size 1.27 1.27)) (justify left))
   )
@@
         )
       )
+    )
+  )
+  (symbol (lib_id "000_Resistors_Immo:100k") (at 169.545 136.525 0) (unit 1)
+    (in_bom yes) (on_board yes) (dnp no) (fields_autoplaced)
+    (property "Reference" "R2" (at 169.545 132.08 0)
+      (effects (font (size 1.27 1.27)))
+    )
+    (property "Value" "100k" (at 169.545 134.62 0)
+      (effects (font (size 1.27 1.27)))
+    )
+    (property "Footprint" "Resistor_SMD:R_0805_2012Metric_Pad1.20x1.40mm_HandSolder" (at 169.545 138.303 0)
+      (effects (font (size 1.27 1.27)) hide)
+    )
+    (property "Datasheet" "~" (at 169.545 136.525 90)
+      (effects (font (size 1.27 1.27)) hide)
+    )
+    (property "JLCpart" "C280020" (at 170.815 139.065 0)
+      (effects (font (size 1.27 1.27)) hide)
+    )
+    (property "Cost" "0.0027" (at 169.545 139.065 0)
+      (effects (font (size 1.27 1.27)) hide)
+    )
+    (pin "1")
+    (pin "2")
+    (instances
+      (project "esp32-faerfly-V2.0"
+        (path "/84b7ad53-68b5-40da-9777-f5bb9a09ecb4/9cdb06a8-babb-4d9b-a75e-e6e2cfc518a0"
+          (reference "R2") (unit 1)
+        )
+      )
