File: esp32-faerfly-V2.0/esp32-faerfly-V2.0.kicad_sch (KiCad schematic)
At the start: 18 parts, among them J1 LiPo_4v2, J3 WS2821b, SW1 SW_SPDT_small, U1 MCP73831-2-OT

Commit message: Updates to V2.0 PCB
Parts:
- removed JP1: I Prog, Jumper:SolderJumper-3_P1.3mm_Open_RoundedPad1.0x1.5mm_NumberLabels, symbol Jumper:SolderJumper_3_Open
- removed JP2: usb/batt, Jumper:SolderJumper-3_P1.3mm_Bridged12_RoundedPad1.0x1.5mm, symbol 000_Connectors_Immo:Jumper_3_Bridged12
- removed R1, R2: 10k, Resistor_SMD:R_0805_2012Metric_Pad1.20x1.40mm_HandSolder, symbol 000_Resistors_Immo:10k
- removed R3: 4k7, Resistor_SMD:R_0805_2012Metric_Pad1.20x1.40mm_HandSolder, symbol 000_Resistors_Immo:4k7
- added J11: WS2821b, 000-edge-connectors-immo:3-pin-edge, symbol 000-edge-connectors-immo:3-pin-edge-touch
- added R3: 2k2, Resistor_SMD:R_0805_2012Metric_Pad1.20x1.40mm_HandSolder, symbol 000_Resistors_Immo:2k2
Connections:
- net BATTERY_POWER: now also J1.A2
- net BATTERY_POWER_BUS: now also SW1.2 (B)
- net GND: now also J11.A1, R3.2
- net USB_POWER: now also SW1.3 (C), J11.A3
- net at U1.5 (PROG): now also R3.1
- new net 3V3_BUS: J11.A2
Other:
- sheet ESP32 ports: added BATT_SNIFF, SCL, SDA; removed none
- note added: "2k2 = ~550mA"
- note added: "Programming Resistor Need multiple & jumpers? Version 2 Note: Nope, all batteries were over 500mA, using with high current draw of WLED smaller batteries are less useful"
- note added: "VERSION 2.0: - Prioritise high current path from - Vin Header to SmartLED header for use in higher power lighting projects"
- note removed: "1 open, 3 open = 10 kohm = 100mA 1 close, 3 open = 4k7 ohm = ~ 250mA 1 open, 3 close = 3k1 ohm = ~ 350mA 1 close , 3 close = 2k4 ogm = ~ 500mA"
- note removed: "Change jumper if omitting battery"
- note removed: "Programming Resistor Need multiple & jumpers?"
- moved on the sheet: SW1
